File: hardware/kicad/bridge.kicad_sch (KiCad schematic)
At the start: 72 parts, among them J3 MOTOR_A, J4 MOTOR_B, J5 MOTOR_C, Q3 IPT015N10N5, Q4 IPT015N10N5, Q5 IPT015N10N5, Q6 IPT015N10N5, Q7 IPT015N10N5, Q8 IPT015N10N5, U4 LM5109BMA, U5 INA240A2D, U6 LM5109BMA, U7 INA240A2D, U8 LM5109BMA, U9 INA240A2D

Commit message: Rev B: fix power terminals and design-review findings
Layout (hand-placed power stage):
- BAT+/BAT- and MOTOR A/B/C are now M5 plated bolt terminals at the board
  edges (battery 36 mm apart on the left edge, motors under their shunts),
  replacing 5x10 mm SMD solder pads that sat 7.5 mm apart
- per phase: driver | high FET over low FET (drain tabs up, compact switch
  node) | Kelvin shunt + INA240; DC-link ceramics at the low-side sources
- FET NTC moved next to the middle low-side FET
- rule area keeps tracks off the inner planes under the power stage
- pours sized from real TOLL pad outlines; solid plane connections
- hand route for the one connection Freerouting leaves open; routing
  session saved so the board rebuilds without the autorouter
- KiCad DRC: 0 violations, 0 unconnected, footprints match library

Schematic / firmware:
- INA240A2 -> INA240A1: the 80 A hard trip was above the old +/-66 A ADC
  full scale and could never fire; compile-time assert + sim test added
- 4-terminal Kelvin shunts (BVR 4026) feed the INA240 sense inputs
- gate resistors 10R -> 4R7, bulk caps 6 -> 8

Co-Authored-By: Claude Opus 5.5 <noreply@anthropic.com>
Claude-Session: https://claude.ai/code/session_01KE5bAkgcicsoh5erUtagKE
Parts:
- added C45: 1n, Capacitor_SMD:C_0603_1608Metric, symbol Device:C
- added C46: 100n, Capacitor_SMD:C_0603_1608Metric, symbol Device:C
- C25, C26: value 2.2u/100V -> 220u/100V; footprint Capacitor_SMD:C_1210_3225Metric -> Capacitor_THT:CP_Radial_D12.5mm_P5.00mm; symbol Device:C -> Device:C_Polarized; MPN (none) -> Panasonic EEU-FS2A221 (or eq. low-ESR)
- C31: value 10n -> 2.2u/100V; footprint Capacitor_SMD:C_0603_1608Metric -> Capacitor_SMD:C_1210_3225Metric
- C32: value 1u/25V -> 2.2u/100V; footprint Capacitor_SMD:C_0805_2012Metric -> Capacitor_SMD:C_1210_3225Metric
- C33: value 2.2u/25V -> 10n; footprint Capacitor_SMD:C_0805_2012Metric -> Capacitor_SMD:C_0603_1608Metric
- C34, C38, C42: value 100n -> 1u/25V; footprint Capacitor_SMD:C_0603_1608Metric -> Capacitor_SMD:C_0805_2012Metric
- C35, C39, C43: value 1n -> 2.2u/25V; footprint Capacitor_SMD:C_0603_1608Metric -> Capacitor_SMD:C_0805_2012Metric
- C36, C40: value 1u/25V -> 100n; footprint Capacitor_SMD:C_0805_2012Metric -> Capacitor_SMD:C_0603_1608Metric
- C37, C41: value 2.2u/25V -> 1n; footprint Capacitor_SMD:C_0805_2012Metric -> Capacitor_SMD:C_0603_1608Metric
- J3, J4, J5: footprint Connector_Wire:SolderWirePad_1x01_SMD_5x10mm -> MountingHole:MountingHole_5.3mm_M5_Pad_Via; MPN (none) -> M5 ring lug terminal
- R22, R24, R30, R32, R38, R40: value 10R -> 4R7
- R26, R34, R42: footprint Resistor_SMD:R_2512_6332Metric -> Resistor_SMD:R_Shunt_Isabellenhuette_BVR4026; symbol Device:R -> Device:R_Shunt; MPN Bourns CRA2512-FZ-R500ELF (3 W) -> Isabellenhuette BVR 4026, 0.5 mOhm, 5 W
- U5, U7, U9: value INA240A2D -> INA240A1D; symbol Amplifier_Current:INA240A2D -> Amplifier_Current:INA240A1D
Connections:
- net +12V: now also C34.1, C38.1, C42.1; no longer C32.1, C36.1, C40.1
- net +3V3: now also C36.1, C40.1, C44.1; no longer C34.1, C38.1, C42.1
- net +48V: now also C31.1, C32.1
- net GND: now also C33.2, C37.2, C41.2, C45.2, C46.2; no longer C35.2, C39.2, C43.2
- net HB_A: now also C35.1; no longer C33.1
- net HB_B: now also C39.1; no longer C37.1
- net HB_C: now also C43.1; no longer C41.1
- net ISENSE_A: now also C37.1; no longer C35.1
- net ISENSE_B: now also C41.1; no longer C39.1
- net ISENSE_C: now also C45.1; no longer C43.1
- net PHASE_A: now also R26.4; no longer R26.2, U5.1 (-)
- net PHASE_B: now also R34.4; no longer R34.2, U7.1 (-)
- net PHASE_C: now also R42.4; no longer R42.2, U9.1 (-)
- net SW_A: now also C35.2; no longer C33.2, U5.8 (+)
- net SW_B: now also C39.2; no longer C37.2, U7.8 (+)
- net SW_C: now also C43.2; no longer C41.2, U9.8 (+)
- net TEMP_FET: now also C46.1; no longer C44.1
- net VBUS_SENSE: now also C33.1; no longer C31.1
- new net ISN_A: R26.3, U5.1 (-)
- new net ISN_B: R34.3, U7.1 (-)
- new net ISN_C: R42.3, U9.1 (-)
- new net ISP_A: R26.2, U5.8 (+)
- new net ISP_B: R34.2, U7.8 (+)
- new net ISP_C: R42.2, U9.8 (+)
Other:
- moved on the sheet: C31, C32, C33, C34, C35, C36, C37, C38, C39, C40, C41, C42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

Commit message: Rev C: compact 188x74 mm layout, re-routed, DRC clean; JLCPCB cost notes
- Repack the power stage into 38 mm phase columns and the logic into a 52 mm
  strip; smaller SRN8040TA buck inductors
- Re-route with Freerouting; record the LATCH_B hand route and move
  references that land on neighbouring silkscreen
- Regenerate BOM, schematic PDF, layer images and 3D renders (stand-in model
  for the SRN8040TA)
- README: rev C notes, phase-pour current capacity, JLCPCB cost estimate

Co-Authored-By: Claude Opus 5.5 <noreply@anthropic.com>
Claude-Session: https://claude.ai/code/session_01KE5bAkgcicsoh5erUtagKE
Parts:
- C19, C20, C21, C22, C23, C24, C25, C26: MPN Panasonic EEU-FS2A221 (or eq. low-ESR) -> Panasonic EEU-FS2A221 or eq. low-ESR, >=2.1 A ripple
Changed lines of the file:
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@@
     (property "Footprint" "Capacitor_THT:CP_Radial_D12.5mm_P5.00mm" (at 17.78 38.1 0) (effects (font (size 1.27 1.27)) hide))
     (property "Datasheet" "~" (at 17.78 38.1 0) (effects (font (size 1.27 1.27)) hide))
-    (property "MPN" "Panasonic EEU-FS2A221 (or eq. low-ESR)" (at 17.78 38.1 0) (effects (font (size 1.27 1.27)) hide))
+    (property "MPN" "Panasonic EEU-FS2A221 or eq. low-ESR, >=2.1 A ripple" (at 17.78 38.1 0) (effects (font (size 1.27 1.27)) hide))
     (pin "1")
     (pin "2")
@@
     (property "Footprint" "Capacitor_THT:CP_Radial_D12.5mm_P5.00mm" (at 33.02 38.1 0) (effects (font (size 1.27 1.27)) hide))
     (property "Datasheet" "~" (at 33.02 38.1 0) (effects (font (size 1.27 1.27)) hide))
-    (property "MPN" "Panasonic EEU-FS2A221 (or eq. low-ESR)" (at 33.02 38.1 0) (effects (font (size 1.27 1.27)) hide))
+    (property "MPN" "Panasonic EEU-FS2A221 or eq. low-ESR, >=2.1 A ripple" (at 33.02 38.1 0) (effects (font (size 1.27 1.27)) hide))
     (pin "1")
     (pin "2")
@@
     (property "Footprint" "Capacitor_THT:CP_Radial_D12.5mm_P5.00mm" (at 48.26 38.1 0) (effects (font (size 1.27 1.27)) hide))
     (property "Datasheet" "~" (at 48.26 38.1 0) (effects (font (size 1.27 1.27)) hide))
-    (property "MPN" "Panasonic EEU-FS2A221 (or eq. low-ESR)" (at 48.26 38.1 0) (effects (font (size 1.27 1.27)) hide))
+    (property "MPN" "Panasonic EEU-FS2A221 or eq. low-ESR, >=2.1 A ripple" (at 48.26 38.1 0) (effects (font (size 1.27 1.27)) hide))
     (pin "1")
     (pin "2")
@@
     (property "Footprint" "Capacitor_THT:CP_Radial_D12.5mm_P5.00mm" (at 63.5 38.1 0) (effects (font (size 1.27 1.27)) hide))
     (property "Datasheet" "~" (at 63.5 38.1 0) (effects (font (size 1.27 1.27)) hide))
-    (property "MPN" "Panasonic EEU-FS2A221 (or eq. low-ESR)" (at 63.5 38.1 0) (effects (font (size 1.27 1.27)) hide))
+    (property "MPN" "Panasonic EEU-FS2A221 or eq. low-ESR, >=2.1 A ripple" (at 63.5 38.1 0) (effects (font (size 1.27 1.27)) hide))
     (pin "1")
     (pin "2")
@@
     (property "Footprint" "Capacitor_THT:CP_Radial_D12.5mm_P5.00mm" (at 78.74 38.1 0) (effects (font (size 1.27 1.27)) hide))
     (property "Datasheet" "~" (at 78.74 38.1 0) (effects (font (size 1.27 1.27)) hide))
-    (property "MPN" "Panasonic EEU-FS2A221 (or eq. low-ESR)" (at 78.74 38.1 0) (effects (font (size 1.27 1.27)) hide))
+    (property "MPN" "Panasonic EEU-FS2A221 or eq. low-ESR, >=2.1 A ripple" (at 78.74 38.1 0) (effects (font (size 1.27 1.27)) hide))
     (pin "1")
     (pin "2")
@@
     (property "Footprint" "Capacitor_THT:CP_Radial_D12.5mm_P5.00mm" (at 93.98 38.1 0) (effects (font (size 1.27 1.27)) hide))
     (property "Datasheet" "~" (at 93.98 38.1 0) (effects (font (size 1.27 1.27)) hide))
-    (property "MPN" "Panasonic EEU-FS2A221 (or eq. low-ESR)" (at 93.98 38.1 0) (effects (font (size 1.27 1.27)) hide))
+    (property "MPN" "Panasonic EEU-FS2A221 or eq. low-ESR, >=2.1 A ripple" (at 93.98 38.1 0) (effects (font (size 1.27 1.27)) hide))
     (pin "1")
     (pin "2")
@@
     (property "Footprint" "Capacitor_THT:CP_Radial_D12.5mm_P5.00mm" (at 109.22 38.1 0) (effects (font (size 1.27 1.27)) hide))
     (property "Datasheet" "~" (at 109.22 38.1 0) (effects (font (size 1.27 1.27)) hide))
-    (property "MPN" "Panasonic EEU-FS2A221 (or eq. low-ESR)" (at 109.22 38.1 0) (effects (font (size 1.27 1.27)) hide))
+    (property "MPN" "Panasonic EEU-FS2A221 or eq. low-ESR, >=2.1 A ripple" (at 109.22 38.1 0) (effects (font (size 1.27 1.27)) hide))
     (pin "1")
     (pin "2")
@@
     (property "Footprint" "Capacitor_THT:CP_Radial_D12.5mm_P5.00mm" (at 124.46 38.1 0) (effects (font (size 1.27 1.27)) hide))
     (property "Datasheet" "~" (at 124.46 38.1 0) (effects (font (size 1.27 1.27)) hide))
-    (property "MPN" "Panasonic EEU-FS2A221 (or eq. low-ESR)" (at 124.46 38.1 0) (effects (font (size 1.27 1.27)) hide))
-    (pin "1")
-    (pin "2")
+    (property "MPN" "Panasonic EEU-FS2A221 or eq. low-ESR, >=2.1 A ripple" (at 124.46 38.1 0) (effects (font (size 1.27 1.27)) hide))
+    (pin "1")
+    (pin "2")

Commit message: BOM: Bourns CSS4J-4026R-L500F as the JLCPCB-stocked shunt
Co-Authored-By: Claude Opus 5.5 <noreply@anthropic.com>
Claude-Session: https://claude.ai/code/session_01KE5bAkgcicsoh5erUtagKE
Parts:
- R26, R34, R42: MPN Isabellenhuette BVR 4026, 0.5 mOhm, 5 W -> Bourns CSS4J-4026R-L500F (LCSC C2076423) or Isabellenhuette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
Changed lines of the file:
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@@
     (property "Footprint" "Resistor_SMD:R_Shunt_Isabellenhuette_BVR4026" (at 83.82 88.9 0) (effects (font (size 1.27 1.27)) hide))
     (property "Datasheet" "~" (at 83.82 88.9 0) (effects (font (size 1.27 1.27)) hide))
-    (property "MPN" "Isabellenhuette BVR 4026, 0.5 mOhm, 5 W" (at 83.82 88.9 0) (effects (font (size 1.27 1.27)) hide))
+    (property "MPN" "Bourns CSS4J-4026R-L500F (LCSC C2076423) or Isabellenhuette BVR 4026; 0.5 mOhm 1% 5 W" (at 83.82 88.9 0) (effects (font (size 1.27 1.27)) hide))
     (pin "1")
     (pin "2")
@@
     (property "Footprint" "Resistor_SMD:R_Shunt_Isabellenhuette_BVR4026" (at 17.78 134.62 0) (effects (font (size 1.27 1.27)) hide))
     (property "Datasheet" "~" (at 17.78 134.62 0) (effects (font (size 1.27 1.27)) hide))
-    (property "MPN" "Isabellenhuette BVR 4026, 0.5 mOhm, 5 W" (at 17.78 134.62 0) (effects (font (size 1.27 1.27)) hide))
+    (property "MPN" "Bourns CSS4J-4026R-L500F (LCSC C2076423) or Isabellenhuette BVR 4026; 0.5 mOhm 1% 5 W" (at 17.78 134.62 0) (effects (font (size 1.27 1.27)) hide))
     (pin "1")
     (pin "2")
@@
     (property "Footprint" "Resistor_SMD:R_Shunt_Isabellenhuette_BVR4026" (at 342.9 134.62 0) (effects (font (size 1.27 1.27)) hide))
     (property "Datasheet" "~" (at 342.9 134.62 0) (effects (font (size 1.27 1.27)) hide))
-    (property "MPN" "Isabellenhuette BVR 4026, 0.5 mOhm, 5 W" (at 342.9 134.62 0) (effects (font (size 1.27 1.27)) hide))
-    (pin "1")
-    (pin "2")
+    (property "MPN" "Bourns CSS4J-4026R-L500F (LCSC C2076423) or Isabellenhuette BVR 4026; 0.5 mOhm 1% 5 W" (at 342.9 134.62 0) (effects (font (size 1.27 1.27)) hide))
+    (pin "1")
+    (pin "2")

Commit message: Use Bourns CSS4J-4026R-L500F shunts (JLCPCB C2076423)
Same 0.5 mOhm / 1 % / 5 W and land pattern as the BVR 4026 footprint, so the
layout and firmware scaling are unchanged. Update the cost estimate.

Co-Authored-By: Claude Opus 5.5 <noreply@anthropic.com>
Claude-Session: https://claude.ai/code/session_01KE5bAkgcicsoh5erUtagKE
Parts:
- R26, R34, R42: MPN Bourns CSS4J-4026R-L500F (LCSC C2076423) or Isabellenhuette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 -> Bourns CSS4J-4026R-L500F (LCSC C2076423), 0.5 mOhm 1% 5 W
Changed lines of the file:
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@@
     (property "Footprint" "Resistor_SMD:R_Shunt_Isabellenhuette_BVR4026" (at 83.82 88.9 0) (effects (font (size 1.27 1.27)) hide))
     (property "Datasheet" "~" (at 83.82 88.9 0) (effects (font (size 1.27 1.27)) hide))
-    (property "MPN" "Bourns CSS4J-4026R-L500F (LCSC C2076423) or Isabellenhuette BVR 4026; 0.5 mOhm 1% 5 W" (at 83.82 88.9 0) (effects (font (size 1.27 1.27)) hide))
+    (property "MPN" "Bourns CSS4J-4026R-L500F (LCSC C2076423), 0.5 mOhm 1% 5 W" (at 83.82 88.9 0) (effects (font (size 1.27 1.27)) hide))
     (pin "1")
     (pin "2")
@@
     (property "Footprint" "Resistor_SMD:R_Shunt_Isabellenhuette_BVR4026" (at 17.78 134.62 0) (effects (font (size 1.27 1.27)) hide))
     (property "Datasheet" "~" (at 17.78 134.62 0) (effects (font (size 1.27 1.27)) hide))
-    (property "MPN" "Bourns CSS4J-4026R-L500F (LCSC C2076423) or Isabellenhuette BVR 4026; 0.5 mOhm 1% 5 W" (at 17.78 134.62 0) (effects (font (size 1.27 1.27)) hide))
+    (property "MPN" "Bourns CSS4J-4026R-L500F (LCSC C2076423), 0.5 mOhm 1% 5 W" (at 17.78 134.62 0) (effects (font (size 1.27 1.27)) hide))
     (pin "1")
     (pin "2")
@@
     (property "Footprint" "Resistor_SMD:R_Shunt_Isabellenhuette_BVR4026" (at 342.9 134.62 0) (effects (font (size 1.27 1.27)) hide))
     (property "Datasheet" "~" (at 342.9 134.62 0) (effects (font (size 1.27 1.27)) hide))
-    (property "MPN" "Bourns CSS4J-4026R-L500F (LCSC C2076423) or Isabellenhuette BVR 4026; 0.5 mOhm 1% 5 W" (at 342.9 134.62 0) (effects (font (size 1.27 1.27)) hide))
-    (pin "1")
-    (pin "2")
+    (property "MPN" "Bourns CSS4J-4026R-L500F (LCSC C2076423), 0.5 mOhm 1% 5 W" (at 342.9 134.62 0) (effects (font (size 1.27 1.27)) hide))
+    (pin "1")
+    (pin "2")

Commit message: BOM: LCSC part numbers, replacements for unstocked parts; revise cost
Bulk 220 uF/100 V caps are not stocked at LCSC: buy separately or use global
sourcing. Add a stocked alternative for the 33 uH inductor. Fix the cost
total (the low end did not match the sum of the rows).

Co-Authored-By: Claude Opus 5.5 <noreply@anthropic.com>
Claude-Session: https://claude.ai/code/session_01KE5bAkgcicsoh5erUtagKE
Parts:
- C19, C20, C21, C22, C23, C24, C25, C26: MPN Panasonic EEU-FS2A221 or eq. low-ESR, >=2.1 A ripple -> Panasonic EEU-FS2A221 or Rubycon 100ZLH220MEFC12.5X25 (12.5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
- TH1: MPN NCP18XH103F03RB -> Murata NCP18XH103F03RB (LCSC C13564)
Changed lines of the file:
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@@
     (property "Footprint" "Capacitor_THT:CP_Radial_D12.5mm_P5.00mm" (at 17.78 38.1 0) (effects (font (size 1.27 1.27)) hide))
     (property "Datasheet" "~" (at 17.78 38.1 0) (effects (font (size 1.27 1.27)) hide))
-    (property "MPN" "Panasonic EEU-FS2A221 or eq. low-ESR, >=2.1 A ripple" (at 17.78 38.1 0) (effects (font (size 1.27 1.27)) hide))
+    (property "MPN" "Panasonic EEU-FS2A221 or Rubycon 100ZLH220MEFC12.5X25 (12.5x25 mm, 5 mm pitch, low-ESR); not stocked at LCSC: global sourcing or hand-solder" (at 17.78 38.1 0) (effects (font (size 1.27 1.27)) hide))
     (pin "1")
     (pin "2")
@@
     (property "Footprint" "Capacitor_THT:CP_Radial_D12.5mm_P5.00mm" (at 33.02 38.1 0) (effects (font (size 1.27 1.27)) hide))
     (property "Datasheet" "~" (at 33.02 38.1 0) (effects (font (size 1.27 1.27)) hide))
-    (property "MPN" "Panasonic EEU-FS2A221 or eq. low-ESR, >=2.1 A ripple" (at 33.02 38.1 0) (effects (font (size 1.27 1.27)) hide))
+    (property "MPN" "Panasonic EEU-FS2A221 or Rubycon 100ZLH220MEFC12.5X25 (12.5x25 mm, 5 mm pitch, low-ESR); not stocked at LCSC: global sourcing or hand-solder" (at 33.02 38.1 0) (effects (font (size 1.27 1.27)) hide))
     (pin "1")
     (pin "2")
@@
     (property "Footprint" "Capacitor_THT:CP_Radial_D12.5mm_P5.00mm" (at 48.26 38.1 0) (effects (font (size 1.27 1.27)) hide))
     (property "Datasheet" "~" (at 48.26 38.1 0) (effects (font (size 1.27 1.27)) hide))
-    (property "MPN" "Panasonic EEU-FS2A221 or eq. low-ESR, >=2.1 A ripple" (at 48.26 38.1 0) (effects (font (size 1.27 1.27)) hide))
+    (property "MPN" "Panasonic EEU-FS2A221 or Rubycon 100ZLH220MEFC12.5X25 (12.5x25 mm, 5 mm pitch, low-ESR); not stocked at LCSC: global sourcing or hand-solder" (at 48.26 38.1 0) (effects (font (size 1.27 1.27)) hide))
     (pin "1")
     (pin "2")
@@
     (property "Footprint" "Capacitor_THT:CP_Radial_D12.5mm_P5.00mm" (at 63.5 38.1 0) (effects (font (size 1.27 1.27)) hide))
     (property "Datasheet" "~" (at 63.5 38.1 0) (effects (font (size 1.27 1.27)) hide))
-    (property "MPN" "Panasonic EEU-FS2A221 or eq. low-ESR, >=2.1 A ripple" (at 63.5 38.1 0) (effects (font (size 1.27 1.27)) hide))
+    (property "MPN" "Panasonic EEU-FS2A221 or Rubycon 100ZLH220MEFC12.5X25 (12.5x25 mm, 5 mm pitch, low-ESR); not stocked at LCSC: global sourcing or hand-solder" (at 63.5 38.1 0) (effects (font (size 1.27 1.27)) hide))
     (pin "1")
     (pin "2")
@@
     (property "Footprint" "Capacitor_THT:CP_Radial_D12.5mm_P5.00mm" (at 78.74 38.1 0) (effects (font (size 1.27 1.27)) hide))
     (property "Datasheet" "~" (at 78.74 38.1 0) (effects (font (size 1.27 1.27)) hide))
-    (property "MPN" "Panasonic EEU-FS2A221 or eq. low-ESR, >=2.1 A ripple" (at 78.74 38.1 0) (effects (font (size 1.27 1.27)) hide))
+    (property "MPN" "Panasonic EEU-FS2A221 or Rubycon 100ZLH220MEFC12.5X25 (12.5x25 mm, 5 mm pitch, low-ESR); not stocked at LCSC: global sourcing or hand-solder" (at 78.74 38.1 0) (effects (font (size 1.27 1.27)) hide))
     (pin "1")
     (pin "2")
@@
     (property "Footprint" "Capacitor_THT:CP_Radial_D12.5mm_P5.00mm" (at 93.98 38.1 0) (effects (font (size 1.27 1.27)) hide))
     (property "Datasheet" "~" (at 93.98 38.1 0) (effects (font (size 1.27 1.27)) hide))
-    (property "MPN" "Panasonic EEU-FS2A221 or eq. low-ESR, >=2.1 A ripple" (at 93.98 38.1 0) (effects (font (size 1.27 1.27)) hide))
+    (property "MPN" "Panasonic EEU-FS2A221 or Rubycon 100ZLH220MEFC12.5X25 (12.5x25 mm, 5 mm pitch, low-ESR); not stocked at LCSC: global sourcing or hand-solder" (at 93.98 38.1 0) (effects (font (size 1.27 1.27)) hide))
     (pin "1")
     (pin "2")
@@
     (property "Footprint" "Capacitor_THT:CP_Radial_D12.5mm_P5.00mm" (at 109.22 38.1 0) (effects (font (size 1.27 1.27)) hide))
     (property "Datasheet" "~" (at 109.22 38.1 0) (effects (font (size 1.27 1.27)) hide))
-    (property "MPN" "Panasonic EEU-FS2A221 or eq. low-ESR, >=2.1 A ripple" (at 109.22 38.1 0) (effects (font (size 1.27 1.27)) hide))
+    (property "MPN" "Panasonic EEU-FS2A221 or Rubycon 100ZLH220MEFC12.5X25 (12.5x25 mm, 5 mm pitch, low-ESR); not stocked at LCSC: global sourcing or hand-solder" (at 109.22 38.1 0) (effects (font (size 1.27 1.27)) hide))
     (pin "1")
     (pin "2")
@@
     (property "Footprint" "Capacitor_THT:CP_Radial_D12.5mm_P5.00mm" (at 124.46 38.1 0) (effects (font (size 1.27 1.27)) hide))
     (property "Datasheet" "~" (at 124.46 38.1 0) (effects (font (size 1.27 1.27)) hide))
-    (property "MPN" "Panasonic EEU-FS2A221 or eq. low-ESR, >=2.1 A ripple" (at 124.46 38.1 0) (effects (font (size 1.27 1.27)) hide))
+    (property "MPN" "Panasonic EEU-FS2A221 or Rubycon 100ZLH220MEFC12.5X25 (12.5x25 mm, 5 mm pitch, low-ESR); not stocked at LCSC: global sourcing or hand-solder" (at 124.46 38.1 0) (effects (font (size 1.27 1.27)) hide))
     (pin "1")
     (pin "2")
@@
     (property "Footprint" "Resistor_SMD:R_0603_1608Metric" (at 73.66 185.42 0) (effects (font (size 1.27 1.27)) hide))
     (property "Datasheet" "~" (at 73.66 185.42 0) (effects (font (size 1.27 1.27)) hide))
-    (property "MPN" "NCP18XH103F03RB" (at 73.66 185.42 0) (effects (font (size 1.27 1.27)) hide))
-    (pin "1")
-    (pin "2")
+    (property "MPN" "Murata NCP18XH103F03RB (LCSC C13564)" (at 73.66 185.42 0) (effects (font (size 1.27 1.27)) hide))
+    (pin "1")
+    (pin "2")
