File: hardware/kicad/bridge.kicad_sch (KiCad schematic)
At the start: 74 parts, among them J3 MOTOR_A, J4 MOTOR_B, J5 MOTOR_C, Q3 IPT015N10N5, Q4 IPT015N10N5, Q5 IPT015N10N5, Q6 IPT015N10N5, Q7 IPT015N10N5, Q8 IPT015N10N5, U4 LM5109BMA, U5 INA240A1D, U6 LM5109BMA, U7 INA240A1D, U8 LM5109BMA, U9 INA240A1D

Commit message: Rev D (in progress): compact placement tooling, stocked bulk caps
- Skyline packer with 90-degree rotation for small parts (fills regions
  far better than the row packer)
- Fix reference-overlap check: SWIG proxies are never identical, so every
  reference was compared with itself and hidden
- Rev D geometry: 185 x 66 mm, motor terminals beside the DC-link ceramics,
  narrower battery strip (board file stays rev C until routing is done)
- Bulk caps: Aishi ERS1KM221W25OT (LCSC C106684)

Co-Authored-By: Claude Opus 5.5 <noreply@anthropic.com>
Claude-Session: https://claude.ai/code/session_01KE5bAkgcicsoh5erUtagKE
Parts:
- C19, C20, C21, C22, C23, C24, C25, C26: MPN Panasonic EEU-FS2A221 or Rubycon 100ZLH220MEFC12.5X25 (12.5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 -> Aishi ERS1KM221W25OT (LCSC C106684), 12.5x25 mm, 5 mm pitch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
Changed lines of the file:
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@@
     (property "Footprint" "Capacitor_THT:CP_Radial_D12.5mm_P5.00mm" (at 17.78 38.1 0) (effects (font (size 1.27 1.27)) hide))
     (property "Datasheet" "~" (at 17.78 38.1 0) (effects (font (size 1.27 1.27)) hide))
-    (property "MPN" "Panasonic EEU-FS2A221 or Rubycon 100ZLH220MEFC12.5X25 (12.5x25 mm, 5 mm pitch, low-ESR); not stocked at LCSC: global sourcing or hand-solder" (at 17.78 38.1 0) (effects (font (size 1.27 1.27)) hide))
+    (property "MPN" "Aishi ERS1KM221W25OT (LCSC C106684), 12.5x25 mm, 5 mm pitch; alt. Panasonic EEU-FS2A221" (at 17.78 38.1 0) (effects (font (size 1.27 1.27)) hide))
     (pin "1")
     (pin "2")
@@
     (property "Footprint" "Capacitor_THT:CP_Radial_D12.5mm_P5.00mm" (at 33.02 38.1 0) (effects (font (size 1.27 1.27)) hide))
     (property "Datasheet" "~" (at 33.02 38.1 0) (effects (font (size 1.27 1.27)) hide))
-    (property "MPN" "Panasonic EEU-FS2A221 or Rubycon 100ZLH220MEFC12.5X25 (12.5x25 mm, 5 mm pitch, low-ESR); not stocked at LCSC: global sourcing or hand-solder" (at 33.02 38.1 0) (effects (font (size 1.27 1.27)) hide))
+    (property "MPN" "Aishi ERS1KM221W25OT (LCSC C106684), 12.5x25 mm, 5 mm pitch; alt. Panasonic EEU-FS2A221" (at 33.02 38.1 0) (effects (font (size 1.27 1.27)) hide))
     (pin "1")
     (pin "2")
@@
     (property "Footprint" "Capacitor_THT:CP_Radial_D12.5mm_P5.00mm" (at 48.26 38.1 0) (effects (font (size 1.27 1.27)) hide))
     (property "Datasheet" "~" (at 48.26 38.1 0) (effects (font (size 1.27 1.27)) hide))
-    (property "MPN" "Panasonic EEU-FS2A221 or Rubycon 100ZLH220MEFC12.5X25 (12.5x25 mm, 5 mm pitch, low-ESR); not stocked at LCSC: global sourcing or hand-solder" (at 48.26 38.1 0) (effects (font (size 1.27 1.27)) hide))
+    (property "MPN" "Aishi ERS1KM221W25OT (LCSC C106684), 12.5x25 mm, 5 mm pitch; alt. Panasonic EEU-FS2A221" (at 48.26 38.1 0) (effects (font (size 1.27 1.27)) hide))
     (pin "1")
     (pin "2")
@@
     (property "Footprint" "Capacitor_THT:CP_Radial_D12.5mm_P5.00mm" (at 63.5 38.1 0) (effects (font (size 1.27 1.27)) hide))
     (property "Datasheet" "~" (at 63.5 38.1 0) (effects (font (size 1.27 1.27)) hide))
-    (property "MPN" "Panasonic EEU-FS2A221 or Rubycon 100ZLH220MEFC12.5X25 (12.5x25 mm, 5 mm pitch, low-ESR); not stocked at LCSC: global sourcing or hand-solder" (at 63.5 38.1 0) (effects (font (size 1.27 1.27)) hide))
+    (property "MPN" "Aishi ERS1KM221W25OT (LCSC C106684), 12.5x25 mm, 5 mm pitch; alt. Panasonic EEU-FS2A221" (at 63.5 38.1 0) (effects (font (size 1.27 1.27)) hide))
     (pin "1")
     (pin "2")
@@
     (property "Footprint" "Capacitor_THT:CP_Radial_D12.5mm_P5.00mm" (at 78.74 38.1 0) (effects (font (size 1.27 1.27)) hide))
     (property "Datasheet" "~" (at 78.74 38.1 0) (effects (font (size 1.27 1.27)) hide))
-    (property "MPN" "Panasonic EEU-FS2A221 or Rubycon 100ZLH220MEFC12.5X25 (12.5x25 mm, 5 mm pitch, low-ESR); not stocked at LCSC: global sourcing or hand-solder" (at 78.74 38.1 0) (effects (font (size 1.27 1.27)) hide))
+    (property "MPN" "Aishi ERS1KM221W25OT (LCSC C106684), 12.5x25 mm, 5 mm pitch; alt. Panasonic EEU-FS2A221" (at 78.74 38.1 0) (effects (font (size 1.27 1.27)) hide))
     (pin "1")
     (pin "2")
@@
     (property "Footprint" "Capacitor_THT:CP_Radial_D12.5mm_P5.00mm" (at 93.98 38.1 0) (effects (font (size 1.27 1.27)) hide))
     (property "Datasheet" "~" (at 93.98 38.1 0) (effects (font (size 1.27 1.27)) hide))
-    (property "MPN" "Panasonic EEU-FS2A221 or Rubycon 100ZLH220MEFC12.5X25 (12.5x25 mm, 5 mm pitch, low-ESR); not stocked at LCSC: global sourcing or hand-solder" (at 93.98 38.1 0) (effects (font (size 1.27 1.27)) hide))
+    (property "MPN" "Aishi ERS1KM221W25OT (LCSC C106684), 12.5x25 mm, 5 mm pitch; alt. Panasonic EEU-FS2A221" (at 93.98 38.1 0) (effects (font (size 1.27 1.27)) hide))
     (pin "1")
     (pin "2")
@@
     (property "Footprint" "Capacitor_THT:CP_Radial_D12.5mm_P5.00mm" (at 109.22 38.1 0) (effects (font (size 1.27 1.27)) hide))
     (property "Datasheet" "~" (at 109.22 38.1 0) (effects (font (size 1.27 1.27)) hide))
-    (property "MPN" "Panasonic EEU-FS2A221 or Rubycon 100ZLH220MEFC12.5X25 (12.5x25 mm, 5 mm pitch, low-ESR); not stocked at LCSC: global sourcing or hand-solder" (at 109.22 38.1 0) (effects (font (size 1.27 1.27)) hide))
+    (property "MPN" "Aishi ERS1KM221W25OT (LCSC C106684), 12.5x25 mm, 5 mm pitch; alt. Panasonic EEU-FS2A221" (at 109.22 38.1 0) (effects (font (size 1.27 1.27)) hide))
     (pin "1")
     (pin "2")
@@
     (property "Footprint" "Capacitor_THT:CP_Radial_D12.5mm_P5.00mm" (at 124.46 38.1 0) (effects (font (size 1.27 1.27)) hide))
     (property "Datasheet" "~" (at 124.46 38.1 0) (effects (font (size 1.27 1.27)) hide))
-    (property "MPN" "Panasonic EEU-FS2A221 or Rubycon 100ZLH220MEFC12.5X25 (12.5x25 mm, 5 mm pitch, low-ESR); not stocked at LCSC: global sourcing or hand-solder" (at 124.46 38.1 0) (effects (font (size 1.27 1.27)) hide))
-    (pin "1")
-    (pin "2")
+    (property "MPN" "Aishi ERS1KM221W25OT (LCSC C106684), 12.5x25 mm, 5 mm pitch; alt. Panasonic EEU-FS2A221" (at 124.46 38.1 0) (effects (font (size 1.27 1.27)) hide))
+    (pin "1")
+    (pin "2")

Commit message: Rev E: four 1000 uF/100 V bulk caps, 180 x 69.5 mm, routed, DRC clean
- 4 x Aishi ERS1KM102M35OT (LCSC C724666, 18 x 35 mm) spread over the
  bridges instead of 8 x 220 uF: 4000 uF, half the parts
- Rerouted (100 passes); the one open INA240 supply tap closed with a route
  from the new astar_route.py grid router, ending on a via into the +3V3 plane
- RIP_UP drops a 139 mm Freerouting detour on the phase C low-side gate drive;
  it is re-made locally (24 mm, like phases A/B). All phase and switch-node
  pours verified as one piece on both outer layers
- Stand-in 3D model for the 18 mm cans; new renders, layers, BOM, PDF, README

Co-Authored-By: Claude Opus 5.5 <noreply@anthropic.com>
Claude-Session: https://claude.ai/code/session_01KE5bAkgcicsoh5erUtagKE
Parts:
- removed C43: 2.2u/25V, Capacitor_SMD:C_0805_2012Metric, symbol Device:C
- removed C44, C46: 100n, Capacitor_SMD:C_0603_1608Metric, symbol Device:C
- removed C45: 1n, Capacitor_SMD:C_0603_1608Metric, symbol Device:C
- C19, C20, C21, C22: value 220u/100V -> 1000u/100V; footprint Capacitor_THT:CP_Radial_D12.5mm_P5.00mm -> Capacitor_THT:CP_Radial_D18.0mm_P7.50mm; MPN Aishi ERS1KM221W25OT (LCSC C106684), 12.5x25 mm, 5 mm pitch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 -> Aishi ERS1KM102M35OT (LCSC C724666), 18x35 mm, 7.5 mm pitch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
- C23, C24, C25, C26: value 220u/100V -> 2.2u/100V; footprint Capacitor_THT:CP_Radial_D12.5mm_P5.00mm -> Capacitor_SMD:C_1210_3225Metric; symbol Device:C_Polarized -> Device:C; MPN Aishi ERS1KM221W25OT (LCSC C106684), 12.5x25 mm, 5 mm pitch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 -> (none)
- C29: value 2.2u/100V -> 10n; footprint Capacitor_SMD:C_1210_3225Metric -> Capacitor_SMD:C_0603_1608Metric
- C30: value 2.2u/100V -> 1u/25V; footprint Capacitor_SMD:C_1210_3225Metric -> Capacitor_SMD:C_0805_2012Metric
- C31: value 2.2u/100V -> 2.2u/25V; footprint Capacitor_SMD:C_1210_3225Metric -> Capacitor_SMD:C_0805_2012Metric
- C32: value 2.2u/100V -> 100n; footprint Capacitor_SMD:C_1210_3225Metric -> Capacitor_SMD:C_0603_1608Metric
- C33: value 10n -> 1n
- C42: value 1u/25V -> 100n; footprint Capacitor_SMD:C_0805_2012Metric -> Capacitor_SMD:C_0603_1608Metric
Connections:
- net +12V: now also C30.1; no longer C42.1
- net +3V3: now also C32.1
- net +48V: no longer C29.1, C30.1, C31.1, C32.1
- net GND: no longer C31.2
- net HB_A: now also C31.1; no longer C35.1
- net HB_B: now also C35.1; no longer C39.1
- net HB_C: now also C39.1
- net ISENSE_A: now also C33.1; no longer C37.1
- net ISENSE_B: now also C37.1; no longer C41.1
- net ISENSE_C: now also C41.1
- net SW_A: now also C31.2; no longer C35.2
- net SW_B: now also C35.2; no longer C39.2
- net SW_C: now also C39.2
- net TEMP_FET: now also C42.1
- net VBUS_SENSE: now also C29.1; no longer C33.1
Other:
- moved on the sheet: C20, C21, C22, C27, C28, C29, C30, C31, C32, C33, C34, C35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

Commit message: Rev F (in progress): DRV8353RS redesign for a 90 x 64.5 mm board
- Circuit: DRV8353RS gate driver + CSAs + 5 V buck replaces 3x LM5109B,
  3x INA240 and both LM5164s; low-side Kelvin shunts; 12 AWG solder-wire
  pads; JST-GH connectors; 3x 1000 uF bulk caps; project symbol/footprint
  library (DRV8353RS symbol + TI RGZ footprint from flatmcu, MIT)
- Firmware: SPI1 driver for the DRV8353 (config + readback + lock, fault
  readout, 'drv' command), ADC sampling at the PWM peak via TIM1 TRGO2,
  high-duty phase rebuilt from the other two, DRIVER fault; sim models the
  low-side shunt blind window and a driver fault - all checks pass
- Placement for the two-sided 3-column layout; router keepouts, pours and
  planes for it (board file stays rev E until routing is done)

Co-Authored-By: Claude Opus 5.5 <noreply@anthropic.com>
Claude-Session: https://claude.ai/code/session_01KE5bAkgcicsoh5erUtagKE
Parts:
- removed C35, C39: 2.2u/25V, Capacitor_SMD:C_0805_2012Metric, symbol Device:C
- removed C36, C40, C42: 100n, Capacitor_SMD:C_0603_1608Metric, symbol Device:C
- removed C37, C41: 1n, Capacitor_SMD:C_0603_1608Metric, symbol Device:C
- removed C38: 1u/25V, Capacitor_SMD:C_0805_2012Metric, symbol Device:C
- removed D5, D6, D7: ES1D, Diode_SMD:D_SMA, symbol Device:D
- removed R26, R34, R42: 0.5m, Resistor_SMD:R_Shunt_Isabellenhuette_BVR4026, symbol Device:R_Shunt
- removed R27, R35, R43: 100R, Resistor_SMD:R_0603_1608Metric, symbol Device:R
- removed R28, R29, R31, R33, R36, R37, R39, R41, R44: 10k, Resistor_SMD:R_0603_1608Metric, symbol Device:R
- removed R30, R32, R38, R40: 4R7, Resistor_SMD:R_0603_1608Metric, symbol Device:R
- removed U4, U6, U8: LM5109BMA, Package_SO:SOIC-8_3.9x4.9mm_P1.27mm, symbol Driver_FET:LM5109BMA
- removed U5, U7, U9: INA240A1D, Package_SO:SOIC-8_3.9x4.9mm_P1.27mm, symbol Amplifier_Current:INA240A1D
- added C11, C12, C13: 1000u/100V, Capacitor_THT:CP_Radial_D18.0mm_P7.50mm, symbol Device:C_Polarized
- added C14, C15, C16, C17, C18: 2.2u/100V, Capacitor_SMD:C_1210_3225Metric, symbol Device:C
- added R13: 100k, Resistor_SMD:R_0603_1608Metric, symbol Device:R
- added R14: 5.6k, Resistor_SMD:R_0603_1608Metric, symbol Device:R
- added R15, R17: 10k, Resistor_SMD:R_0603_1608Metric, symbol Device:R
- added R16: 4.7k, Resistor_SMD:R_0603_1608Metric, symbol Device:R
- added U2: DRV8353RS, bldc48:TI-RGZ-48-QFN, symbol bldc48:DRV8353RS
- C19, C22: value 1000u/100V -> 2.2u/100V; footprint Capacitor_THT:CP_Radial_D18.0mm_P7.50mm -> Capacitor_SMD:C_1210_3225Metric; symbol Device:C_Polarized -> Device:C; MPN Aishi ERS1KM102M35OT (LCSC C724666), 18x35 mm, 7.5 mm pitch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 -> (none)
- C20: value 1000u/100V -> 10n; footprint Capacitor_THT:CP_Radial_D18.0mm_P7.50mm -> Capacitor_SMD:C_0603_1608Metric; symbol Device:C_Polarized -> Device:C; MPN Aishi ERS1KM102M35OT (LCSC C724666), 18x35 mm, 7.5 mm pitch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 -> (none)
- C21: value 1000u/100V -> 100n/100V; footprint Capacitor_THT:CP_Radial_D18.0mm_P7.50mm -> Capacitor_SMD:C_0805_2012Metric; symbol Device:C_Polarized -> Device:C; MPN Aishi ERS1KM102M35OT (LCSC C724666), 18x35 mm, 7.5 mm pitch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 -> (none)
- C23: value 2.2u/100V -> 47n/100V; footprint Capacitor_SMD:C_1210_3225Metric -> Capacitor_SMD:C_0805_2012Metric
- C24, C25: value 2.2u/100V -> 1u/16V; footprint Capacitor_SMD:C_1210_3225Metric -> Capacitor_SMD:C_0603_1608Metric
- C26: value 2.2u/100V -> 1u; footprint Capacitor_SMD:C_1210_3225Metric -> Capacitor_SMD:C_0603_1608Metric
- C27: value 2.2u/100V -> 100n; footprint Capacitor_SMD:C_1210_3225Metric -> Capacitor_SMD:C_0603_1608Metric
- C28: value 2.2u/100V -> 1n; footprint Capacitor_SMD:C_1210_3225Metric -> Capacitor_SMD:C_0603_1608Metric
- C29: value 10n -> 1n
- C30: value 1u/25V -> 1n; footprint Capacitor_SMD:C_0805_2012Metric -> Capacitor_SMD:C_0603_1608Metric
- C31: value 2.2u/25V -> 1n; footprint Capacitor_SMD:C_0805_2012Metric -> Capacitor_SMD:C_0603_1608Metric
- C32: value 100n -> 1n
- C34: value 1u/25V -> 100n; footprint Capacitor_SMD:C_0805_2012Metric -> Capacitor_SMD:C_0603_1608Metric
- J3, J4, J5: footprint MountingHole:MountingHole_5.3mm_M5_Pad_Via -> bldc48:SolderWire_12AWG_D2.8mm_OD5.4mm; MPN M5 ring lug terminal -> 12 AWG wire, soldered
- R19: value 5.6k -> 0.5m; footprint Resistor_SMD:R_0603_1608Metric -> Resistor_SMD:R_Shunt_Isabellenhuette_BVR4026; symbol Device:R -> Device:R_Shunt; MPN (none) -> Bourns CSS4J-4026R-L500F (LCSC C2076423), 0.5 mOhm 1% 5 W
- R20: value 10k -> 100R
- R21, R23: value 10k -> 0.5m; footprint Resistor_SMD:R_0603_1608Metric -> Resistor_SMD:R_Shunt_Isabellenhuette_BVR4026; symbol Device:R -> Device:R_Shunt; MPN (none) -> Bourns CSS4J-4026R-L500F (LCSC C2076423), 0.5 mOhm 1% 5 W
- R22, R24: value 4R7 -> 100R
Connections:
- net HB_A is gone; now on net ISENSE_B: C31.1
- net PHASE_A is gone; now on net SW_A: J3.1 (Pin_1)
- net PHASE_B is gone; now on net SW_B: J4.1 (Pin_1)
- net PHASE_C is gone; now on net SW_C: J5.1 (Pin_1)
- net +3V3: now also C27.1, R25.1, R15.1, R16.1, R17.1, U2.26 (VREF); no longer C32.1
- net +48V: now also C24.2, C11.1, C12.1, C13.1, C14.1, C15.1, C16.1, C17.1, C18.1, R13.1, U2.43 (VIN), U2.5 (VM), U2.6 (VDRAIN); no longer C20.1, C23.1, C24.1, C25.1, C26.1, C27.1, C28.1, R18.1
- net GH_A: now also U2.8 (GHA); no longer R22.2, R23.1
- net GH_B: now also U2.17 (GHB)
- net GH_C: now also U2.18 (GHC)
- net GL_A: now also U2.10 (GLA); no longer R24.2, R25.1
- net GL_B: now also U2.15 (GLB)
- net GL_C: now also U2.20 (GLC)
- net GND: now also C31.2, R18.2, R19.4, R21.4, R23.4, C11.2, C12.2, C13.2, C14.2, C15.2, C16.2, C17.2, C18.2, R14.2, U2.1 (GND), U2.27 (AGND), U2.41 (DGND), U2.49 (PAD); no longer C23.2, C24.2, C28.2, C30.2, C32.2, Q4.2 (S), Q6.2 (S), Q8.2 (S), R19.2, R20.2, R21.2, R25.2
- net ISENSE_A: now also C29.1, R20.2; no longer C33.1
- net ISENSE_B: now also R22.2
- net ISENSE_C: now also C33.1, R24.2
- net PWM_AH: now also U2.34 (INHA); no longer R20.1
- net PWM_AL: now also U2.35 (INLA); no longer R21.1
- net PWM_BH: now also U2.36 (INHB)
- net PWM_BL: now also U2.37 (INLB)
- net PWM_CH: now also U2.38 (INHC)
- net PWM_CL: now also U2.39 (INLC)
- net SW_A: now also U2.9 (SHA); no longer C31.2, R23.2
- net SW_B: now also U2.16 (SHB)
- net SW_C: now also U2.19 (SHC)
- net TEMP_FET: now also C34.1, R25.2
- net VBUS_SENSE: now also C20.1, R13.2, R14.1; no longer C29.1, R18.2, R19.1
- net +12V renamed SP_B
- net SP_B: now also R21.2, U2.14 (SPB); no longer C34.1
- net HO_A renamed SO_B
- net SO_B: now also U2.24 (SOB)
- net LO_A renamed SO_C
- net SO_C: now also U2.23 (SOC)
- new net BST5: U2.45 (BST)
- new net CPH: C23.2, U2.4 (CPH)
- new net CPL: C23.1, U2.3 (CPL)
- new net DRV_CS: R17.2, U2.32 (nSCS)
- new net DRV_EN: R18.1, U2.33 (ENABLE)
- new net DRV_FAULT: R15.2, U2.28 (nFAULT)
- new net DRV_SCK: U2.31 (SCLK)
- new net DRV_SDI: U2.30 (SDI)
- new net DRV_SDO: R16.2, U2.29 (SDO)
- new net DVDD: C26.1, U2.40 (DVDD)
- new net FB5: U2.48 (FB)
- new net LS_A: Q4.2 (S), R19.1
- new net LS_B: Q6.2 (S), R21.1
- new net LS_C: Q8.2 (S), R23.1
- new net RCL: U2.46 (RCL)
- new net RT_SD: U2.47 (RT/SD)
- new net SN_A: C28.2, R19.3, U2.12 (SNA)
- new net SN_B: C30.2, R21.3, U2.13 (SNB)
- new net SN_C: C32.2, R23.3, U2.22 (SNC)
- new net SO_A: R20.1, U2.25 (SOA)
- new net SP_A: C28.1, R19.2, U2.11 (SPA)
- new net SP_C: C32.1, R23.2, U2.21 (SPC)
- new net SW5: U2.42 (SW)
- new net VCC_B: U2.44 (VCC)
- new net VCP: C24.1, U2.7 (VCP)
- new net VGLS: C25.1, U2.2 (VGLS)
Other:
- note added: "DRV8353RS gate driver, 3-phase power stage, low-side current sensing"
- note removed: "3-phase power stage and current sensing"
- title: 3-phase power stage and current sensing -> DRV8353RS gate driver, 3-phase power stage, low-side current sensing
- moved on the sheet: C23, C24, C25, C26, C27, C28, C29, C30, C31, C32, C33, C34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
