File: hardware/kicad/io.kicad_sch (KiCad schematic)
At the start: 36 parts, among them J10 BRAKE, J11 POWER_BTN, J12 UART, J7 HALL, J8 THROTTLE, J9 FWD/REV

Commit message: Rev B: fix power terminals and design-review findings
Layout (hand-placed power stage):
- BAT+/BAT- and MOTOR A/B/C are now M5 plated bolt terminals at the board
  edges (battery 36 mm apart on the left edge, motors under their shunts),
  replacing 5x10 mm SMD solder pads that sat 7.5 mm apart
- per phase: driver | high FET over low FET (drain tabs up, compact switch
  node) | Kelvin shunt + INA240; DC-link ceramics at the low-side sources
- FET NTC moved next to the middle low-side FET
- rule area keeps tracks off the inner planes under the power stage
- pours sized from real TOLL pad outlines; solid plane connections
- hand route for the one connection Freerouting leaves open; routing
  session saved so the board rebuilds without the autorouter
- KiCad DRC: 0 violations, 0 unconnected, footprints match library

Schematic / firmware:
- INA240A2 -> INA240A1: the 80 A hard trip was above the old +/-66 A ADC
  full scale and could never fire; compile-time assert + sim test added
- 4-terminal Kelvin shunts (BVR 4026) feed the INA240 sense inputs
- gate resistors 10R -> 4R7, bulk caps 6 -> 8

Co-Authored-By: Claude Opus 5.5 <noreply@anthropic.com>
Claude-Session: https://claude.ai/code/session_01KE5bAkgcicsoh5erUtagKE
Parts:
- removed C53, C54: 1n, Capacitor_SMD:C_0603_1608Metric, symbol Device:C
- added C60, C61: 100n, Capacitor_SMD:C_0603_1608Metric, symbol Device:C
- C56, C57: value 100n -> 1n
Connections:
- net BRAKE: now also C61.1; no longer C59.1
- net DIR_SW: now also C60.1; no longer C58.1
- net GND: now also C60.2, C61.2
- net HALL_A: now also C55.1
- net HALL_B: now also C56.1
- net HALL_C: now also C57.1; no longer C55.1
- net TEMP_MOTOR: now also C58.1; no longer C56.1
- net THROTTLE: now also C59.1; no longer C57.1
Other:
- moved on the sheet: C55, C56, C57, C58, C59
Changed lines of the file:
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@@
     (rev "A")
     (company "48V 35A hub motor controller")
-    (comment 1 "STM32G431 + LM5109B x3 + IPT015N10N5 x6 + INA240A2 x3")
+    (comment 1 "STM32G431 + LM5109B x3 + IPT015N10N5 x6 + INA240A1 x3")
     (comment 2 "Sheet: io")
   )
@@
   (symbol (lib_id "Device:C") (at 66.04 43.18 0) (unit 1)
     (in_bom yes) (on_board yes) (dnp no)
-    (property "Reference" "C53" (at 69.072 38.37 0) (effects (font (size 1.27 1.27)) (justify left)))
+    (property "Reference" "C55" (at 69.072 38.37 0) (effects (font (size 1.27 1.27)) (justify left)))
     (property "Value" "1n" (at 69.072 48.99 0) (effects (font (size 1.27 1.27)) (justify left)))
     (property "Footprint" "Capacitor_SMD:C_0603_1608Metric" (at 66.04 43.18 0) (effects (font (size 1.27 1.27)) hide))
@@
     (pin "1")
     (pin "2")
-    (instances (project "bldc48" (path "/1b798bf4-fe80-550a-af47-9df77e3c6d45/0dd75bc2-a6c8-5971-a840-21b6a986b1c7" (reference "C53") (unit 1))))
+    (instances (project "bldc48" (path "/1b798bf4-fe80-550a-af47-9df77e3c6d45/0dd75bc2-a6c8-5971-a840-21b6a986b1c7" (reference "C55") (unit 1))))
   )
   (wire (pts (xy 66.04 39.37) (xy 66.04 36.83)) (stroke (width 0) (type default)))
@@
   (symbol (lib_id "Device:C") (at 96.52 43.18 0) (unit 1)
     (in_bom yes) (on_board yes) (dnp no)
-    (property "Reference" "C54" (at 99.552 38.37 0) (effects (font (size 1.27 1.27)) (justify left)))
+    (property "Reference" "C56" (at 99.552 38.37 0) (effects (font (size 1.27 1.27)) (justify left)))
     (property "Value" "1n" (at 99.552 48.99 0) (effects (font (size 1.27 1.27)) (justify left)))
     (property "Footprint" "Capacitor_SMD:C_0603_1608Metric" (at 96.52 43.18 0) (effects (font (size 1.27 1.27)) hide))
@@
     (pin "1")
     (pin "2")
-    (instances (project "bldc48" (path "/1b798bf4-fe80-550a-af47-9df77e3c6d45/0dd75bc2-a6c8-5971-a840-21b6a986b1c7" (reference "C54") (unit 1))))
+    (instances (project "bldc48" (path "/1b798bf4-fe80-550a-af47-9df77e3c6d45/0dd75bc2-a6c8-5971-a840-21b6a986b1c7" (reference "C56") (unit 1))))
   )
   (wire (pts (xy 96.52 39.37) (xy 96.52 36.83)) (stroke (width 0) (type default)))
@@
   (symbol (lib_id "Device:C") (at 127 43.18 0) (unit 1)
     (in_bom yes) (on_board yes) (dnp no)
-    (property "Reference" "C55" (at 130.032 38.37 0) (effects (font (size 1.27 1.27)) (justify left)))
+    (property "Reference" "C57" (at 130.032 38.37 0) (effects (font (size 1.27 1.27)) (justify left)))
     (property "Value" "1n" (at 130.032 48.99 0) (effects (font (size 1.27 1.27)) (justify left)))
     (property "Footprint" "Capacitor_SMD:C_0603_1608Metric" (at 127 43.18 0) (effects (font (size 1.27 1.27)) hide))
@@
     (pin "1")
     (pin "2")
-    (instances (project "bldc48" (path "/1b798bf4-fe80-550a-af47-9df77e3c6d45/0dd75bc2-a6c8-5971-a840-21b6a986b1c7" (reference "C55") (unit 1))))
+    (instances (project "bldc48" (path "/1b798bf4-fe80-550a-af47-9df77e3c6d45/0dd75bc2-a6c8-5971-a840-21b6a986b1c7" (reference "C57") (unit 1))))
   )
   (wire (pts (xy 127 39.37) (xy 127 36.83)) (stroke (width 0) (type default)))
@@
   (symbol (lib_id "Device:C") (at 157.48 48.26 0) (unit 1)
     (in_bom yes) (on_board yes) (dnp no)
-    (property "Reference" "C56" (at 160.512 43.45 0) (effects (font (size 1.27 1.27)) (justify left)))
+    (property "Reference" "C58" (at 160.512 43.45 0) (effects (font (size 1.27 1.27)) (justify left)))
     (property "Value" "100n" (at 160.512 54.07 0) (effects (font (size 1.27 1.27)) (justify left)))
     (property "Footprint" "Capacitor_SMD:C_0603_1608Metric" (at 157.48 48.26 0) (effects (font (size 1.27 1.27)) hide))
@@
     (pin "1")
     (pin "2")
-    (instances (project "bldc48" (path "/1b798bf4-fe80-550a-af47-9df77e3c6d45/0dd75bc2-a6c8-5971-a840-21b6a986b1c7" (reference "C56") (unit 1))))
+    (instances (project "bldc48" (path "/1b798bf4-fe80-550a-af47-9df77e3c6d45/0dd75bc2-a6c8-5971-a840-21b6a986b1c7" (reference "C58") (unit 1))))
   )
   (wire (pts (xy 157.48 44.45) (xy 157.48 41.91)) (stroke (width 0) (type default)))
@@
   (symbol (lib_id "Device:C") (at 231.14 45.72 0) (unit 1)
     (in_bom yes) (on_board yes) (dnp no)
-    (property "Reference" "C57" (at 234.172 40.91 0) (effects (font (size 1.27 1.27)) (justify left)))
+    (property "Reference" "C59" (at 234.172 40.91 0) (effects (font (size 1.27 1.27)) (justify left)))
     (property "Value" "100n" (at 234.172 51.53 0) (effects (font (size 1.27 1.27)) (justify left)))
     (property "Footprint" "Capacitor_SMD:C_0603_1608Metric" (at 231.14 45.72 0) (effects (font (size 1.27 1.27)) hide))
@@
     (pin "1")
     (pin "2")
-    (instances (project "bldc48" (path "/1b798bf4-fe80-550a-af47-9df77e3c6d45/0dd75bc2-a6c8-5971-a840-21b6a986b1c7" (reference "C57") (unit 1))))
+    (instances (project "bldc48" (path "/1b798bf4-fe80-550a-af47-9df77e3c6d45/0dd75bc2-a6c8-5971-a840-21b6a986b1c7" (reference "C59") (unit 1))))
   )
   (wire (pts (xy 231.14 41.91) (xy 231.14 39.37)) (stroke (width 0) (type default)))
@@
   (symbol (lib_id "Device:C") (at 284.48 43.18 0) (unit 1)
     (in_bom yes) (on_board yes) (dnp no)
-    (property "Reference" "C58" (at 287.512 38.37 0) (effects (font (size 1.27 1.27)) (justify left)))
+    (property "Reference" "C60" (at 287.512 38.37 0) (effects (font (size 1.27 1.27)) (justify left)))
     (property "Value" "100n" (at 287.512 48.99 0) (effects (font (size 1.27 1.27)) (justify left)))
     (property "Footprint" "Capacitor_SMD:C_0603_1608Metric" (at 284.48 43.18 0) (effects (font (size 1.27 1.27)) hide))
@@
     (pin "1")
     (pin "2")
-    (instances (project "bldc48" (path "/1b798bf4-fe80-550a-af47-9df77e3c6d45/0dd75bc2-a6c8-5971-a840-21b6a986b1c7" (reference "C58") (unit 1))))
+    (instances (project "bldc48" (path "/1b798bf4-fe80-550a-af47-9df77e3c6d45/0dd75bc2-a6c8-5971-a840-21b6a986b1c7" (reference "C60") (unit 1))))
   )
   (wire (pts (xy 284.48 39.37) (xy 284.48 36.83)) (stroke (width 0) (type default)))
@@
   (symbol (lib_id "Device:C") (at 340.36 43.18 0) (unit 1)
     (in_bom yes) (on_board yes) (dnp no)
-    (property "Reference" "C59" (at 343.392 38.37 0) (effects (font (size 1.27 1.27)) (justify left)))
+    (property "Reference" "C61" (at 343.392 38.37 0) (effects (font (size 1.27 1.27)) (justify left)))
     (property "Value" "100n" (at 343.392 48.99 0) (effects (font (size 1.27 1.27)) (justify left)))
     (property "Footprint" "Capacitor_SMD:C_0603_1608Metric" (at 340.36 43.18 0) (effects (font (size 1.27 1.27)) hide))
@@
     (pin "1")
     (pin "2")
-    (instances (project "bldc48" (path "/1b798bf4-fe80-550a-af47-9df77e3c6d45/0dd75bc2-a6c8-5971-a840-21b6a986b1c7" (reference "C59") (unit 1))))
+    (instances (project "bldc48" (path "/1b798bf4-fe80-550a-af47-9df77e3c6d45/0dd75bc2-a6c8-5971-a840-21b6a986b1c7" (reference "C61") (unit 1))))
   )
   (wire (pts (xy 340.36 39.37) (xy 340.36 36.83)) (stroke (width 0) (type default)))

Commit message: Rev E: four 1000 uF/100 V bulk caps, 180 x 69.5 mm, routed, DRC clean
- 4 x Aishi ERS1KM102M35OT (LCSC C724666, 18 x 35 mm) spread over the
  bridges instead of 8 x 220 uF: 4000 uF, half the parts
- Rerouted (100 passes); the one open INA240 supply tap closed with a route
  from the new astar_route.py grid router, ending on a via into the +3V3 plane
- RIP_UP drops a 139 mm Freerouting detour on the phase C low-side gate drive;
  it is re-made locally (24 mm, like phases A/B). All phase and switch-node
  pours verified as one piece on both outer layers
- Stand-in 3D model for the 18 mm cans; new renders, layers, BOM, PDF, README

Co-Authored-By: Claude Opus 5.5 <noreply@anthropic.com>
Claude-Session: https://claude.ai/code/session_01KE5bAkgcicsoh5erUtagKE
Parts:
- removed C58, C59, C60, C61: 100n, Capacitor_SMD:C_0603_1608Metric, symbol Device:C
- added C51, C52, C53: 1n, Capacitor_SMD:C_0603_1608Metric, symbol Device:C
- added C54: 100n, Capacitor_SMD:C_0603_1608Metric, symbol Device:C
- C55, C56, C57: value 1n -> 100n
Connections:
- net BRAKE: now also C57.1
- net DIR_SW: now also C56.1
- net GND: now also C51.2, C52.2, C53.2, C54.2
- net HALL_A: now also C51.1; no longer C55.1
- net HALL_B: now also C52.1; no longer C56.1
- net HALL_C: now also C53.1; no longer C57.1
- net TEMP_MOTOR: now also C54.1
- net THROTTLE: now also C55.1
Other:
- moved on the sheet: C55, C56, C57
Changed lines of the file:
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@@
   (symbol (lib_id "Device:C") (at 66.04 43.18 0) (unit 1)
     (in_bom yes) (on_board yes) (dnp no)
-    (property "Reference" "C55" (at 69.072 38.37 0) (effects (font (size 1.27 1.27)) (justify left)))
+    (property "Reference" "C51" (at 69.072 38.37 0) (effects (font (size 1.27 1.27)) (justify left)))
     (property "Value" "1n" (at 69.072 48.99 0) (effects (font (size 1.27 1.27)) (justify left)))
     (property "Footprint" "Capacitor_SMD:C_0603_1608Metric" (at 66.04 43.18 0) (effects (font (size 1.27 1.27)) hide))
@@
     (pin "1")
     (pin "2")
-    (instances (project "bldc48" (path "/1b798bf4-fe80-550a-af47-9df77e3c6d45/0dd75bc2-a6c8-5971-a840-21b6a986b1c7" (reference "C55") (unit 1))))
+    (instances (project "bldc48" (path "/1b798bf4-fe80-550a-af47-9df77e3c6d45/0dd75bc2-a6c8-5971-a840-21b6a986b1c7" (reference "C51") (unit 1))))
   )
   (wire (pts (xy 66.04 39.37) (xy 66.04 36.83)) (stroke (width 0) (type default)))
@@
   (symbol (lib_id "Device:C") (at 96.52 43.18 0) (unit 1)
     (in_bom yes) (on_board yes) (dnp no)
-    (property "Reference" "C56" (at 99.552 38.37 0) (effects (font (size 1.27 1.27)) (justify left)))
+    (property "Reference" "C52" (at 99.552 38.37 0) (effects (font (size 1.27 1.27)) (justify left)))
     (property "Value" "1n" (at 99.552 48.99 0) (effects (font (size 1.27 1.27)) (justify left)))
     (property "Footprint" "Capacitor_SMD:C_0603_1608Metric" (at 96.52 43.18 0) (effects (font (size 1.27 1.27)) hide))
@@
     (pin "1")
     (pin "2")
-    (instances (project "bldc48" (path "/1b798bf4-fe80-550a-af47-9df77e3c6d45/0dd75bc2-a6c8-5971-a840-21b6a986b1c7" (reference "C56") (unit 1))))
+    (instances (project "bldc48" (path "/1b798bf4-fe80-550a-af47-9df77e3c6d45/0dd75bc2-a6c8-5971-a840-21b6a986b1c7" (reference "C52") (unit 1))))
   )
   (wire (pts (xy 96.52 39.37) (xy 96.52 36.83)) (stroke (width 0) (type default)))
@@
   (symbol (lib_id "Device:C") (at 127 43.18 0) (unit 1)
     (in_bom yes) (on_board yes) (dnp no)
-    (property "Reference" "C57" (at 130.032 38.37 0) (effects (font (size 1.27 1.27)) (justify left)))
+    (property "Reference" "C53" (at 130.032 38.37 0) (effects (font (size 1.27 1.27)) (justify left)))
     (property "Value" "1n" (at 130.032 48.99 0) (effects (font (size 1.27 1.27)) (justify left)))
     (property "Footprint" "Capacitor_SMD:C_0603_1608Metric" (at 127 43.18 0) (effects (font (size 1.27 1.27)) hide))
@@
     (pin "1")
     (pin "2")
-    (instances (project "bldc48" (path "/1b798bf4-fe80-550a-af47-9df77e3c6d45/0dd75bc2-a6c8-5971-a840-21b6a986b1c7" (reference "C57") (unit 1))))
+    (instances (project "bldc48" (path "/1b798bf4-fe80-550a-af47-9df77e3c6d45/0dd75bc2-a6c8-5971-a840-21b6a986b1c7" (reference "C53") (unit 1))))
   )
   (wire (pts (xy 127 39.37) (xy 127 36.83)) (stroke (width 0) (type default)))
@@
   (symbol (lib_id "Device:C") (at 157.48 48.26 0) (unit 1)
     (in_bom yes) (on_board yes) (dnp no)
-    (property "Reference" "C58" (at 160.512 43.45 0) (effects (font (size 1.27 1.27)) (justify left)))
+    (property "Reference" "C54" (at 160.512 43.45 0) (effects (font (size 1.27 1.27)) (justify left)))
     (property "Value" "100n" (at 160.512 54.07 0) (effects (font (size 1.27 1.27)) (justify left)))
     (property "Footprint" "Capacitor_SMD:C_0603_1608Metric" (at 157.48 48.26 0) (effects (font (size 1.27 1.27)) hide))
@@
     (pin "1")
     (pin "2")
-    (instances (project "bldc48" (path "/1b798bf4-fe80-550a-af47-9df77e3c6d45/0dd75bc2-a6c8-5971-a840-21b6a986b1c7" (reference "C58") (unit 1))))
+    (instances (project "bldc48" (path "/1b798bf4-fe80-550a-af47-9df77e3c6d45/0dd75bc2-a6c8-5971-a840-21b6a986b1c7" (reference "C54") (unit 1))))
   )
   (wire (pts (xy 157.48 44.45) (xy 157.48 41.91)) (stroke (width 0) (type default)))
@@
   (symbol (lib_id "Device:C") (at 231.14 45.72 0) (unit 1)
     (in_bom yes) (on_board yes) (dnp no)
-    (property "Reference" "C59" (at 234.172 40.91 0) (effects (font (size 1.27 1.27)) (justify left)))
+    (property "Reference" "C55" (at 234.172 40.91 0) (effects (font (size 1.27 1.27)) (justify left)))
     (property "Value" "100n" (at 234.172 51.53 0) (effects (font (size 1.27 1.27)) (justify left)))
     (property "Footprint" "Capacitor_SMD:C_0603_1608Metric" (at 231.14 45.72 0) (effects (font (size 1.27 1.27)) hide))
@@
     (pin "1")
     (pin "2")
-    (instances (project "bldc48" (path "/1b798bf4-fe80-550a-af47-9df77e3c6d45/0dd75bc2-a6c8-5971-a840-21b6a986b1c7" (reference "C59") (unit 1))))
+    (instances (project "bldc48" (path "/1b798bf4-fe80-550a-af47-9df77e3c6d45/0dd75bc2-a6c8-5971-a840-21b6a986b1c7" (reference "C55") (unit 1))))
   )
   (wire (pts (xy 231.14 41.91) (xy 231.14 39.37)) (stroke (width 0) (type default)))
@@
   (symbol (lib_id "Device:C") (at 284.48 43.18 0) (unit 1)
     (in_bom yes) (on_board yes) (dnp no)
-    (property "Reference" "C60" (at 287.512 38.37 0) (effects (font (size 1.27 1.27)) (justify left)))
+    (property "Reference" "C56" (at 287.512 38.37 0) (effects (font (size 1.27 1.27)) (justify left)))
     (property "Value" "100n" (at 287.512 48.99 0) (effects (font (size 1.27 1.27)) (justify left)))
     (property "Footprint" "Capacitor_SMD:C_0603_1608Metric" (at 284.48 43.18 0) (effects (font (size 1.27 1.27)) hide))
@@
     (pin "1")
     (pin "2")
-    (instances (project "bldc48" (path "/1b798bf4-fe80-550a-af47-9df77e3c6d45/0dd75bc2-a6c8-5971-a840-21b6a986b1c7" (reference "C60") (unit 1))))
+    (instances (project "bldc48" (path "/1b798bf4-fe80-550a-af47-9df77e3c6d45/0dd75bc2-a6c8-5971-a840-21b6a986b1c7" (reference "C56") (unit 1))))
   )
   (wire (pts (xy 284.48 39.37) (xy 284.48 36.83)) (stroke (width 0) (type default)))
@@
   (symbol (lib_id "Device:C") (at 340.36 43.18 0) (unit 1)
     (in_bom yes) (on_board yes) (dnp no)
-    (property "Reference" "C61" (at 343.392 38.37 0) (effects (font (size 1.27 1.27)) (justify left)))
+    (property "Reference" "C57" (at 343.392 38.37 0) (effects (font (size 1.27 1.27)) (justify left)))
     (property "Value" "100n" (at 343.392 48.99 0) (effects (font (size 1.27 1.27)) (justify left)))
     (property "Footprint" "Capacitor_SMD:C_0603_1608Metric" (at 340.36 43.18 0) (effects (font (size 1.27 1.27)) hide))
@@
     (pin "1")
     (pin "2")
-    (instances (project "bldc48" (path "/1b798bf4-fe80-550a-af47-9df77e3c6d45/0dd75bc2-a6c8-5971-a840-21b6a986b1c7" (reference "C61") (unit 1))))
+    (instances (project "bldc48" (path "/1b798bf4-fe80-550a-af47-9df77e3c6d45/0dd75bc2-a6c8-5971-a840-21b6a986b1c7" (reference "C57") (unit 1))))
   )
   (wire (pts (xy 340.36 39.37) (xy 340.36 36.83)) (stroke (width 0) (type default)))

Commit message: Rev F (in progress): DRV8353RS redesign for a 90 x 64.5 mm board
- Circuit: DRV8353RS gate driver + CSAs + 5 V buck replaces 3x LM5109B,
  3x INA240 and both LM5164s; low-side Kelvin shunts; 12 AWG solder-wire
  pads; JST-GH connectors; 3x 1000 uF bulk caps; project symbol/footprint
  library (DRV8353RS symbol + TI RGZ footprint from flatmcu, MIT)
- Firmware: SPI1 driver for the DRV8353 (config + readback + lock, fault
  readout, 'drv' command), ADC sampling at the PWM peak via TIM1 TRGO2,
  high-duty phase rebuilt from the other two, DRIVER fault; sim models the
  low-side shunt blind window and a driver fault - all checks pass
- Placement for the two-sided 3-column layout; router keepouts, pours and
  planes for it (board file stays rev E until routing is done)

Co-Authored-By: Claude Opus 5.5 <noreply@anthropic.com>
Claude-Session: https://claude.ai/code/session_01KE5bAkgcicsoh5erUtagKE
Parts:
- removed C51, C52, C53: 1n, Capacitor_SMD:C_0603_1608Metric, symbol Device:C
- removed C54, C55, C56, C57: 100n, Capacitor_SMD:C_0603_1608Metric, symbol Device:C
- removed D10, D11: ESDA6V1-5SC6, Package_TO_SOT_SMD:SOT-23-6, symbol Power_Protection:ESDA6V1-5SC6
- removed R48, R50, R52: 2.2k, Resistor_SMD:R_0603_1608Metric, symbol Device:R
- removed R49, R51, R53, R55, R59, R61: 1k, Resistor_SMD:R_0603_1608Metric, symbol Device:R
- removed R54, R58, R60, R64: 10k, Resistor_SMD:R_0603_1608Metric, symbol Device:R
- removed R56: 12k, Resistor_SMD:R_0603_1608Metric, symbol Device:R
- removed R57: 22k, Resistor_SMD:R_0603_1608Metric, symbol Device:R
- removed R62, R63: 100R, Resistor_SMD:R_0603_1608Metric, symbol Device:R
- added C43, C44, C45: 1n, Capacitor_SMD:C_0603_1608Metric, symbol Device:C
- added C46, C47, C48, C49: 100n, Capacitor_SMD:C_0603_1608Metric, symbol Device:C
- added D8, D9: ESDA6V1-5SC6, Package_TO_SOT_SMD:SOT-23-6, symbol Power_Protection:ESDA6V1-5SC6
- added R29, R31, R33: 2.2k, Resistor_SMD:R_0603_1608Metric, symbol Device:R
- added R30, R32, R34, R36, R40, R42: 1k, Resistor_SMD:R_0603_1608Metric, symbol Device:R
- added R35, R39, R41, R45: 10k, Resistor_SMD:R_0603_1608Metric, symbol Device:R
- added R37: 12k, Resistor_SMD:R_0603_1608Metric, symbol Device:R
- added R38: 22k, Resistor_SMD:R_0603_1608Metric, symbol Device:R
- added R43, R44: 100R, Resistor_SMD:R_0603_1608Metric, symbol Device:R
- J10, J11, J9: footprint Connector_JST:JST_PH_B2B-PH-K_1x02_P2.00mm_Vertical -> Connector_JST:JST_GH_BM02B-GHS-TBT_1x02-1MP_P1.25mm_Vertical; MPN (none) -> JST BM02B-GHS-TBT (1.25 mm, latching)
- J12: footprint Connector_JST:JST_PH_B4B-PH-K_1x04_P2.00mm_Vertical -> Connector_JST:JST_GH_BM04B-GHS-TBT_1x04-1MP_P1.25mm_Vertical; MPN (none) -> JST BM04B-GHS-TBT (1.25 mm, latching)
- J7: footprint Connector_JST:JST_PH_B6B-PH-K_1x06_P2.00mm_Vertical -> Connector_JST:JST_GH_BM06B-GHS-TBT_1x06-1MP_P1.25mm_Vertical; MPN (none) -> JST BM06B-GHS-TBT (1.25 mm, latching)
- J8: footprint Connector_JST:JST_PH_B3B-PH-K_1x03_P2.00mm_Vertical -> Connector_JST:JST_GH_BM03B-GHS-TBT_1x03-1MP_P1.25mm_Vertical; MPN (none) -> JST BM03B-GHS-TBT (1.25 mm, latching)
Connections:
- net +3V3: now also R29.1, R31.1, R33.1, R35.1, R39.1, R41.1, R45.1
- net BRAKE: now also C49.1, R41.2, R42.2
- net BRAKE_IN: now also D9.3 (IO2), R42.1
- net DIR_IN: now also D9.1 (IO1), R40.1
- net DIR_SW: now also C48.1, R39.2, R40.2
- net GND: now also C43.2, C44.2, C45.2, C46.2, C47.2, C48.2, C49.2, D8.2 (GND), D9.2 (GND), R38.2
- net HALL_A: now also C43.1, R30.2
- net HALL_A_IN: now also D8.1 (IO1), R29.2, R30.1
- net HALL_B: now also C44.1, R32.2
- net HALL_B_IN: now also D8.3 (IO2), R31.2, R32.1
- net HALL_C: now also C45.1, R34.2
- net HALL_C_IN: now also D8.4 (IO3), R33.2, R34.1
- net MTEMP_IN: now also D8.5 (IO4), R35.2, R36.1
- net PWR_SW: now also D9.4 (IO3)
- net TEMP_MOTOR: now also C46.1, R36.2
- net THROTTLE: now also C47.1, R37.2, R38.1
- net THR_IN: now also D8.6 (IO5), R37.1
- net UART_RX: now also R44.2, R45.2
- net UART_RX_C: now also D9.6 (IO5), R44.1
- net UART_TX: now also R43.1
- net UART_TX_C: now also D9.5 (IO4), R43.2
