File: hardware/kicad/mcu.kicad_sch (KiCad schematic)
At the start: 16 parts, among them J6 SWD, U10 STM32G431CBT6

Commit message: Rev B: fix power terminals and design-review findings
Layout (hand-placed power stage):
- BAT+/BAT- and MOTOR A/B/C are now M5 plated bolt terminals at the board
  edges (battery 36 mm apart on the left edge, motors under their shunts),
  replacing 5x10 mm SMD solder pads that sat 7.5 mm apart
- per phase: driver | high FET over low FET (drain tabs up, compact switch
  node) | Kelvin shunt + INA240; DC-link ceramics at the low-side sources
- FET NTC moved next to the middle low-side FET
- rule area keeps tracks off the inner planes under the power stage
- pours sized from real TOLL pad outlines; solid plane connections
- hand route for the one connection Freerouting leaves open; routing
  session saved so the board rebuilds without the autorouter
- KiCad DRC: 0 violations, 0 unconnected, footprints match library

Schematic / firmware:
- INA240A2 -> INA240A1: the 80 A hard trip was above the old +/-66 A ADC
  full scale and could never fire; compile-time assert + sim test added
- 4-terminal Kelvin shunts (BVR 4026) feed the INA240 sense inputs
- gate resistors 10R -> 4R7, bulk caps 6 -> 8

Co-Authored-By: Claude Opus 5.5 <noreply@anthropic.com>
Claude-Session: https://claude.ai/code/session_01KE5bAkgcicsoh5erUtagKE
Parts:
- removed C45, C46: 100n, Capacitor_SMD:C_0603_1608Metric, symbol Device:C
- added C53, C54: 100n, Capacitor_SMD:C_0603_1608Metric, symbol Device:C
- C49: value 4.7u -> 100n; footprint Capacitor_SMD:C_0805_2012Metric -> Capacitor_SMD:C_0603_1608Metric
- C50: value 1u -> 100n
- C51: value 100n -> 4.7u; footprint Capacitor_SMD:C_0603_1608Metric -> Capacitor_SMD:C_0805_2012Metric
- C52: value 100n -> 1u
Connections:
- net +3V3: now also C50.1, C51.1
- net +3V3A: now also C52.1, C53.1; no longer C50.1, C51.1
- net GND: now also C53.2, C54.2
- net NRST: now also C54.1; no longer C52.1
Other:
- moved on the sheet: C47, C48, C49, C50, C51, C52
Changed lines of the file:
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@@
     (rev "A")
     (company "48V 35A hub motor controller")
-    (comment 1 "STM32G431 + LM5109B x3 + IPT015N10N5 x6 + INA240A2 x3")
+    (comment 1 "STM32G431 + LM5109B x3 + IPT015N10N5 x6 + INA240A1 x3")
     (comment 2 "Sheet: mcu")
   )
@@
   (symbol (lib_id "Device:C") (at 88.9 38.1 0) (unit 1)
     (in_bom yes) (on_board yes) (dnp no)
-    (property "Reference" "C45" (at 91.932 33.29 0) (effects (font (size 1.27 1.27)) (justify left)))
+    (property "Reference" "C47" (at 91.932 33.29 0) (effects (font (size 1.27 1.27)) (justify left)))
     (property "Value" "100n" (at 91.932 43.91 0) (effects (font (size 1.27 1.27)) (justify left)))
     (property "Footprint" "Capacitor_SMD:C_0603_1608Metric" (at 88.9 38.1 0) (effects (font (size 1.27 1.27)) hide))
@@
     (pin "1")
     (pin "2")
-    (instances (project "bldc48" (path "/1b798bf4-fe80-550a-af47-9df77e3c6d45/ec6ab3a5-f2a6-5f08-bbd4-e129b4dd95cb" (reference "C45") (unit 1))))
+    (instances (project "bldc48" (path "/1b798bf4-fe80-550a-af47-9df77e3c6d45/ec6ab3a5-f2a6-5f08-bbd4-e129b4dd95cb" (reference "C47") (unit 1))))
   )
   (wire (pts (xy 88.9 34.29) (xy 88.9 31.75)) (stroke (width 0) (type default)))
@@
   (symbol (lib_id "Device:C") (at 99.06 38.1 0) (unit 1)
     (in_bom yes) (on_board yes) (dnp no)
-    (property "Reference" "C46" (at 102.092 33.29 0) (effects (font (size 1.27 1.27)) (justify left)))
+    (property "Reference" "C48" (at 102.092 33.29 0) (effects (font (size 1.27 1.27)) (justify left)))
     (property "Value" "100n" (at 102.092 43.91 0) (effects (font (size 1.27 1.27)) (justify left)))
     (property "Footprint" "Capacitor_SMD:C_0603_1608Metric" (at 99.06 38.1 0) (effects (font (size 1.27 1.27)) hide))
@@
     (pin "1")
     (pin "2")
-    (instances (project "bldc48" (path "/1b798bf4-fe80-550a-af47-9df77e3c6d45/ec6ab3a5-f2a6-5f08-bbd4-e129b4dd95cb" (reference "C46") (unit 1))))
+    (instances (project "bldc48" (path "/1b798bf4-fe80-550a-af47-9df77e3c6d45/ec6ab3a5-f2a6-5f08-bbd4-e129b4dd95cb" (reference "C48") (unit 1))))
   )
   (wire (pts (xy 99.06 34.29) (xy 99.06 31.75)) (stroke (width 0) (type default)))
@@
   (symbol (lib_id "Device:C") (at 109.22 38.1 0) (unit 1)
     (in_bom yes) (on_board yes) (dnp no)
-    (property "Reference" "C47" (at 112.252 33.29 0) (effects (font (size 1.27 1.27)) (justify left)))
+    (property "Reference" "C49" (at 112.252 33.29 0) (effects (font (size 1.27 1.27)) (justify left)))
     (property "Value" "100n" (at 112.252 43.91 0) (effects (font (size 1.27 1.27)) (justify left)))
     (property "Footprint" "Capacitor_SMD:C_0603_1608Metric" (at 109.22 38.1 0) (effects (font (size 1.27 1.27)) hide))
@@
     (pin "1")
     (pin "2")
-    (instances (project "bldc48" (path "/1b798bf4-fe80-550a-af47-9df77e3c6d45/ec6ab3a5-f2a6-5f08-bbd4-e129b4dd95cb" (reference "C47") (unit 1))))
+    (instances (project "bldc48" (path "/1b798bf4-fe80-550a-af47-9df77e3c6d45/ec6ab3a5-f2a6-5f08-bbd4-e129b4dd95cb" (reference "C49") (unit 1))))
   )
   (wire (pts (xy 109.22 34.29) (xy 109.22 31.75)) (stroke (width 0) (type default)))
@@
   (symbol (lib_id "Device:C") (at 119.38 38.1 0) (unit 1)
     (in_bom yes) (on_board yes) (dnp no)
-    (property "Reference" "C48" (at 122.412 33.29 0) (effects (font (size 1.27 1.27)) (justify left)))
+    (property "Reference" "C50" (at 122.412 33.29 0) (effects (font (size 1.27 1.27)) (justify left)))
     (property "Value" "100n" (at 122.412 43.91 0) (effects (font (size 1.27 1.27)) (justify left)))
     (property "Footprint" "Capacitor_SMD:C_0603_1608Metric" (at 119.38 38.1 0) (effects (font (size 1.27 1.27)) hide))
@@
     (pin "1")
     (pin "2")
-    (instances (project "bldc48" (path "/1b798bf4-fe80-550a-af47-9df77e3c6d45/ec6ab3a5-f2a6-5f08-bbd4-e129b4dd95cb" (reference "C48") (unit 1))))
+    (instances (project "bldc48" (path "/1b798bf4-fe80-550a-af47-9df77e3c6d45/ec6ab3a5-f2a6-5f08-bbd4-e129b4dd95cb" (reference "C50") (unit 1))))
   )
   (wire (pts (xy 119.38 34.29) (xy 119.38 31.75)) (stroke (width 0) (type default)))
@@
   (symbol (lib_id "Device:C") (at 129.54 38.1 0) (unit 1)
     (in_bom yes) (on_board yes) (dnp no)
-    (property "Reference" "C49" (at 132.572 33.29 0) (effects (font (size 1.27 1.27)) (justify left)))
+    (property "Reference" "C51" (at 132.572 33.29 0) (effects (font (size 1.27 1.27)) (justify left)))
     (property "Value" "4.7u" (at 132.572 43.91 0) (effects (font (size 1.27 1.27)) (justify left)))
     (property "Footprint" "Capacitor_SMD:C_0805_2012Metric" (at 129.54 38.1 0) (effects (font (size 1.27 1.27)) hide))
@@
     (pin "1")
     (pin "2")
-    (instances (project "bldc48" (path "/1b798bf4-fe80-550a-af47-9df77e3c6d45/ec6ab3a5-f2a6-5f08-bbd4-e129b4dd95cb" (reference "C49") (unit 1))))
+    (instances (project "bldc48" (path "/1b798bf4-fe80-550a-af47-9df77e3c6d45/ec6ab3a5-f2a6-5f08-bbd4-e129b4dd95cb" (reference "C51") (unit 1))))
   )
   (wire (pts (xy 129.54 34.29) (xy 129.54 31.75)) (stroke (width 0) (type default)))
@@
   (symbol (lib_id "Device:C") (at 157.48 40.64 0) (unit 1)
     (in_bom yes) (on_board yes) (dnp no)
-    (property "Reference" "C50" (at 160.512 35.83 0) (effects (font (size 1.27 1.27)) (justify left)))
+    (property "Reference" "C52" (at 160.512 35.83 0) (effects (font (size 1.27 1.27)) (justify left)))
     (property "Value" "1u" (at 160.512 46.45 0) (effects (font (size 1.27 1.27)) (justify left)))
     (property "Footprint" "Capacitor_SMD:C_0603_1608Metric" (at 157.48 40.64 0) (effects (font (size 1.27 1.27)) hide))
@@
     (pin "1")
     (pin "2")
-    (instances (project "bldc48" (path "/1b798bf4-fe80-550a-af47-9df77e3c6d45/ec6ab3a5-f2a6-5f08-bbd4-e129b4dd95cb" (reference "C50") (unit 1))))
+    (instances (project "bldc48" (path "/1b798bf4-fe80-550a-af47-9df77e3c6d45/ec6ab3a5-f2a6-5f08-bbd4-e129b4dd95cb" (reference "C52") (unit 1))))
   )
   (wire (pts (xy 157.48 36.83) (xy 157.48 34.29)) (stroke (width 0) (type default)))
@@
   (symbol (lib_id "Device:C") (at 167.64 40.64 0) (unit 1)
     (in_bom yes) (on_board yes) (dnp no)
-    (property "Reference" "C51" (at 170.672 35.83 0) (effects (font (size 1.27 1.27)) (justify left)))
+    (property "Reference" "C53" (at 170.672 35.83 0) (effects (font (size 1.27 1.27)) (justify left)))
     (property "Value" "100n" (at 170.672 46.45 0) (effects (font (size 1.27 1.27)) (justify left)))
     (property "Footprint" "Capacitor_SMD:C_0603_1608Metric" (at 167.64 40.64 0) (effects (font (size 1.27 1.27)) hide))
@@
     (pin "1")
     (pin "2")
-    (instances (project "bldc48" (path "/1b798bf4-fe80-550a-af47-9df77e3c6d45/ec6ab3a5-f2a6-5f08-bbd4-e129b4dd95cb" (reference "C51") (unit 1))))
+    (instances (project "bldc48" (path "/1b798bf4-fe80-550a-af47-9df77e3c6d45/ec6ab3a5-f2a6-5f08-bbd4-e129b4dd95cb" (reference "C53") (unit 1))))
   )
   (wire (pts (xy 167.64 36.83) (xy 167.64 34.29)) (stroke (width 0) (type default)))
@@
   (symbol (lib_id "Device:C") (at 193.04 40.64 0) (unit 1)
     (in_bom yes) (on_board yes) (dnp no)
-    (property "Reference" "C52" (at 196.072 35.83 0) (effects (font (size 1.27 1.27)) (justify left)))
+    (property "Reference" "C54" (at 196.072 35.83 0) (effects (font (size 1.27 1.27)) (justify left)))
     (property "Value" "100n" (at 196.072 46.45 0) (effects (font (size 1.27 1.27)) (justify left)))
     (property "Footprint" "Capacitor_SMD:C_0603_1608Metric" (at 193.04 40.64 0) (effects (font (size 1.27 1.27)) hide))
@@
     (pin "1")
     (pin "2")
-    (instances (project "bldc48" (path "/1b798bf4-fe80-550a-af47-9df77e3c6d45/ec6ab3a5-f2a6-5f08-bbd4-e129b4dd95cb" (reference "C52") (unit 1))))
+    (instances (project "bldc48" (path "/1b798bf4-fe80-550a-af47-9df77e3c6d45/ec6ab3a5-f2a6-5f08-bbd4-e129b4dd95cb" (reference "C54") (unit 1))))
   )
   (wire (pts (xy 193.04 36.83) (xy 193.04 34.29)) (stroke (width 0) (type default)))

Commit message: Rev E: four 1000 uF/100 V bulk caps, 180 x 69.5 mm, routed, DRC clean
- 4 x Aishi ERS1KM102M35OT (LCSC C724666, 18 x 35 mm) spread over the
  bridges instead of 8 x 220 uF: 4000 uF, half the parts
- Rerouted (100 passes); the one open INA240 supply tap closed with a route
  from the new astar_route.py grid router, ending on a via into the +3V3 plane
- RIP_UP drops a 139 mm Freerouting detour on the phase C low-side gate drive;
  it is re-made locally (24 mm, like phases A/B). All phase and switch-node
  pours verified as one piece on both outer layers
- Stand-in 3D model for the 18 mm cans; new renders, layers, BOM, PDF, README

Co-Authored-By: Claude Opus 5.5 <noreply@anthropic.com>
Claude-Session: https://claude.ai/code/session_01KE5bAkgcicsoh5erUtagKE
Parts:
- removed C51: 4.7u, Capacitor_SMD:C_0805_2012Metric, symbol Device:C
- removed C52: 1u, Capacitor_SMD:C_0603_1608Metric, symbol Device:C
- removed C53, C54: 100n, Capacitor_SMD:C_0603_1608Metric, symbol Device:C
- added C43, C44, C45, C46: 100n, Capacitor_SMD:C_0603_1608Metric, symbol Device:C
- C47: value 100n -> 4.7u; footprint Capacitor_SMD:C_0603_1608Metric -> Capacitor_SMD:C_0805_2012Metric
- C48: value 100n -> 1u
Connections:
- net +3V3: now also C43.1, C44.1, C45.1, C46.1; no longer C48.1, C49.1, C50.1
- net +3V3A: now also C48.1, C49.1
- net GND: now also C43.2, C44.2, C45.2, C46.2
- net NRST: now also C50.1
Other:
- moved on the sheet: C47, C48, C49, C50
Changed lines of the file:
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@@
   (symbol (lib_id "Device:C") (at 88.9 38.1 0) (unit 1)
     (in_bom yes) (on_board yes) (dnp no)
-    (property "Reference" "C47" (at 91.932 33.29 0) (effects (font (size 1.27 1.27)) (justify left)))
+    (property "Reference" "C43" (at 91.932 33.29 0) (effects (font (size 1.27 1.27)) (justify left)))
     (property "Value" "100n" (at 91.932 43.91 0) (effects (font (size 1.27 1.27)) (justify left)))
     (property "Footprint" "Capacitor_SMD:C_0603_1608Metric" (at 88.9 38.1 0) (effects (font (size 1.27 1.27)) hide))
@@
     (pin "1")
     (pin "2")
-    (instances (project "bldc48" (path "/1b798bf4-fe80-550a-af47-9df77e3c6d45/ec6ab3a5-f2a6-5f08-bbd4-e129b4dd95cb" (reference "C47") (unit 1))))
+    (instances (project "bldc48" (path "/1b798bf4-fe80-550a-af47-9df77e3c6d45/ec6ab3a5-f2a6-5f08-bbd4-e129b4dd95cb" (reference "C43") (unit 1))))
   )
   (wire (pts (xy 88.9 34.29) (xy 88.9 31.75)) (stroke (width 0) (type default)))
@@
   (symbol (lib_id "Device:C") (at 99.06 38.1 0) (unit 1)
     (in_bom yes) (on_board yes) (dnp no)
-    (property "Reference" "C48" (at 102.092 33.29 0) (effects (font (size 1.27 1.27)) (justify left)))
+    (property "Reference" "C44" (at 102.092 33.29 0) (effects (font (size 1.27 1.27)) (justify left)))
     (property "Value" "100n" (at 102.092 43.91 0) (effects (font (size 1.27 1.27)) (justify left)))
     (property "Footprint" "Capacitor_SMD:C_0603_1608Metric" (at 99.06 38.1 0) (effects (font (size 1.27 1.27)) hide))
@@
     (pin "1")
     (pin "2")
-    (instances (project "bldc48" (path "/1b798bf4-fe80-550a-af47-9df77e3c6d45/ec6ab3a5-f2a6-5f08-bbd4-e129b4dd95cb" (reference "C48") (unit 1))))
+    (instances (project "bldc48" (path "/1b798bf4-fe80-550a-af47-9df77e3c6d45/ec6ab3a5-f2a6-5f08-bbd4-e129b4dd95cb" (reference "C44") (unit 1))))
   )
   (wire (pts (xy 99.06 34.29) (xy 99.06 31.75)) (stroke (width 0) (type default)))
@@
   (symbol (lib_id "Device:C") (at 109.22 38.1 0) (unit 1)
     (in_bom yes) (on_board yes) (dnp no)
-    (property "Reference" "C49" (at 112.252 33.29 0) (effects (font (size 1.27 1.27)) (justify left)))
+    (property "Reference" "C45" (at 112.252 33.29 0) (effects (font (size 1.27 1.27)) (justify left)))
     (property "Value" "100n" (at 112.252 43.91 0) (effects (font (size 1.27 1.27)) (justify left)))
     (property "Footprint" "Capacitor_SMD:C_0603_1608Metric" (at 109.22 38.1 0) (effects (font (size 1.27 1.27)) hide))
@@
     (pin "1")
     (pin "2")
-    (instances (project "bldc48" (path "/1b798bf4-fe80-550a-af47-9df77e3c6d45/ec6ab3a5-f2a6-5f08-bbd4-e129b4dd95cb" (reference "C49") (unit 1))))
+    (instances (project "bldc48" (path "/1b798bf4-fe80-550a-af47-9df77e3c6d45/ec6ab3a5-f2a6-5f08-bbd4-e129b4dd95cb" (reference "C45") (unit 1))))
   )
   (wire (pts (xy 109.22 34.29) (xy 109.22 31.75)) (stroke (width 0) (type default)))
@@
   (symbol (lib_id "Device:C") (at 119.38 38.1 0) (unit 1)
     (in_bom yes) (on_board yes) (dnp no)
-    (property "Reference" "C50" (at 122.412 33.29 0) (effects (font (size 1.27 1.27)) (justify left)))
+    (property "Reference" "C46" (at 122.412 33.29 0) (effects (font (size 1.27 1.27)) (justify left)))
     (property "Value" "100n" (at 122.412 43.91 0) (effects (font (size 1.27 1.27)) (justify left)))
     (property "Footprint" "Capacitor_SMD:C_0603_1608Metric" (at 119.38 38.1 0) (effects (font (size 1.27 1.27)) hide))
@@
     (pin "1")
     (pin "2")
-    (instances (project "bldc48" (path "/1b798bf4-fe80-550a-af47-9df77e3c6d45/ec6ab3a5-f2a6-5f08-bbd4-e129b4dd95cb" (reference "C50") (unit 1))))
+    (instances (project "bldc48" (path "/1b798bf4-fe80-550a-af47-9df77e3c6d45/ec6ab3a5-f2a6-5f08-bbd4-e129b4dd95cb" (reference "C46") (unit 1))))
   )
   (wire (pts (xy 119.38 34.29) (xy 119.38 31.75)) (stroke (width 0) (type default)))
@@
   (symbol (lib_id "Device:C") (at 129.54 38.1 0) (unit 1)
     (in_bom yes) (on_board yes) (dnp no)
-    (property "Reference" "C51" (at 132.572 33.29 0) (effects (font (size 1.27 1.27)) (justify left)))
+    (property "Reference" "C47" (at 132.572 33.29 0) (effects (font (size 1.27 1.27)) (justify left)))
     (property "Value" "4.7u" (at 132.572 43.91 0) (effects (font (size 1.27 1.27)) (justify left)))
     (property "Footprint" "Capacitor_SMD:C_0805_2012Metric" (at 129.54 38.1 0) (effects (font (size 1.27 1.27)) hide))
@@
     (pin "1")
     (pin "2")
-    (instances (project "bldc48" (path "/1b798bf4-fe80-550a-af47-9df77e3c6d45/ec6ab3a5-f2a6-5f08-bbd4-e129b4dd95cb" (reference "C51") (unit 1))))
+    (instances (project "bldc48" (path "/1b798bf4-fe80-550a-af47-9df77e3c6d45/ec6ab3a5-f2a6-5f08-bbd4-e129b4dd95cb" (reference "C47") (unit 1))))
   )
   (wire (pts (xy 129.54 34.29) (xy 129.54 31.75)) (stroke (width 0) (type default)))
@@
   (symbol (lib_id "Device:C") (at 157.48 40.64 0) (unit 1)
     (in_bom yes) (on_board yes) (dnp no)
-    (property "Reference" "C52" (at 160.512 35.83 0) (effects (font (size 1.27 1.27)) (justify left)))
+    (property "Reference" "C48" (at 160.512 35.83 0) (effects (font (size 1.27 1.27)) (justify left)))
     (property "Value" "1u" (at 160.512 46.45 0) (effects (font (size 1.27 1.27)) (justify left)))
     (property "Footprint" "Capacitor_SMD:C_0603_1608Metric" (at 157.48 40.64 0) (effects (font (size 1.27 1.27)) hide))
@@
     (pin "1")
     (pin "2")
-    (instances (project "bldc48" (path "/1b798bf4-fe80-550a-af47-9df77e3c6d45/ec6ab3a5-f2a6-5f08-bbd4-e129b4dd95cb" (reference "C52") (unit 1))))
+    (instances (project "bldc48" (path "/1b798bf4-fe80-550a-af47-9df77e3c6d45/ec6ab3a5-f2a6-5f08-bbd4-e129b4dd95cb" (reference "C48") (unit 1))))
   )
   (wire (pts (xy 157.48 36.83) (xy 157.48 34.29)) (stroke (width 0) (type default)))
@@
   (symbol (lib_id "Device:C") (at 167.64 40.64 0) (unit 1)
     (in_bom yes) (on_board yes) (dnp no)
-    (property "Reference" "C53" (at 170.672 35.83 0) (effects (font (size 1.27 1.27)) (justify left)))
+    (property "Reference" "C49" (at 170.672 35.83 0) (effects (font (size 1.27 1.27)) (justify left)))
     (property "Value" "100n" (at 170.672 46.45 0) (effects (font (size 1.27 1.27)) (justify left)))
     (property "Footprint" "Capacitor_SMD:C_0603_1608Metric" (at 167.64 40.64 0) (effects (font (size 1.27 1.27)) hide))
@@
     (pin "1")
     (pin "2")
-    (instances (project "bldc48" (path "/1b798bf4-fe80-550a-af47-9df77e3c6d45/ec6ab3a5-f2a6-5f08-bbd4-e129b4dd95cb" (reference "C53") (unit 1))))
+    (instances (project "bldc48" (path "/1b798bf4-fe80-550a-af47-9df77e3c6d45/ec6ab3a5-f2a6-5f08-bbd4-e129b4dd95cb" (reference "C49") (unit 1))))
   )
   (wire (pts (xy 167.64 36.83) (xy 167.64 34.29)) (stroke (width 0) (type default)))
@@
   (symbol (lib_id "Device:C") (at 193.04 40.64 0) (unit 1)
     (in_bom yes) (on_board yes) (dnp no)
-    (property "Reference" "C54" (at 196.072 35.83 0) (effects (font (size 1.27 1.27)) (justify left)))
+    (property "Reference" "C50" (at 196.072 35.83 0) (effects (font (size 1.27 1.27)) (justify left)))
     (property "Value" "100n" (at 196.072 46.45 0) (effects (font (size 1.27 1.27)) (justify left)))
     (property "Footprint" "Capacitor_SMD:C_0603_1608Metric" (at 193.04 40.64 0) (effects (font (size 1.27 1.27)) hide))
@@
     (pin "1")
     (pin "2")
-    (instances (project "bldc48" (path "/1b798bf4-fe80-550a-af47-9df77e3c6d45/ec6ab3a5-f2a6-5f08-bbd4-e129b4dd95cb" (reference "C54") (unit 1))))
+    (instances (project "bldc48" (path "/1b798bf4-fe80-550a-af47-9df77e3c6d45/ec6ab3a5-f2a6-5f08-bbd4-e129b4dd95cb" (reference "C50") (unit 1))))
   )
   (wire (pts (xy 193.04 36.83) (xy 193.04 34.29)) (stroke (width 0) (type default)))

Commit message: Rev F (in progress): DRV8353RS redesign for a 90 x 64.5 mm board
- Circuit: DRV8353RS gate driver + CSAs + 5 V buck replaces 3x LM5109B,
  3x INA240 and both LM5164s; low-side Kelvin shunts; 12 AWG solder-wire
  pads; JST-GH connectors; 3x 1000 uF bulk caps; project symbol/footprint
  library (DRV8353RS symbol + TI RGZ footprint from flatmcu, MIT)
- Firmware: SPI1 driver for the DRV8353 (config + readback + lock, fault
  readout, 'drv' command), ADC sampling at the PWM peak via TIM1 TRGO2,
  high-duty phase rebuilt from the other two, DRIVER fault; sim models the
  low-side shunt blind window and a driver fault - all checks pass
- Placement for the two-sided 3-column layout; router keepouts, pours and
  planes for it (board file stays rev E until routing is done)

Co-Authored-By: Claude Opus 5.5 <noreply@anthropic.com>
Claude-Session: https://claude.ai/code/session_01KE5bAkgcicsoh5erUtagKE
Parts:
- removed C43, C44, C45, C46, C49, C50: 100n, Capacitor_SMD:C_0603_1608Metric, symbol Device:C
- removed C47: 4.7u, Capacitor_SMD:C_0805_2012Metric, symbol Device:C
- removed C48: 1u, Capacitor_SMD:C_0603_1608Metric, symbol Device:C
- removed D8: GREEN, LED_SMD:LED_0603_1608Metric, symbol Device:LED
- removed D9: RED, LED_SMD:LED_0603_1608Metric, symbol Device:LED
- removed R45: 10k, Resistor_SMD:R_0603_1608Metric, symbol Device:R
- removed R46, R47: 1k, Resistor_SMD:R_0603_1608Metric, symbol Device:R
- removed U10: STM32G431CBT6, Package_QFP:LQFP-48_7x7mm_P0.5mm, symbol MCU_ST_STM32G4:STM32G431CBTx
- added C35, C36, C37, C38, C41, C42: 100n, Capacitor_SMD:C_0603_1608Metric, symbol Device:C
- added C39: 4.7u, Capacitor_SMD:C_0805_2012Metric, symbol Device:C
- added C40: 1u, Capacitor_SMD:C_0603_1608Metric, symbol Device:C
- added D6: GREEN, LED_SMD:LED_0603_1608Metric, symbol Device:LED
- added D7: RED, LED_SMD:LED_0603_1608Metric, symbol Device:LED
- added R26: 10k, Resistor_SMD:R_0603_1608Metric, symbol Device:R
- added R27, R28: 1k, Resistor_SMD:R_0603_1608Metric, symbol Device:R
- added U3: STM32G431CBT6, Package_QFP:LQFP-48_7x7mm_P0.5mm, symbol MCU_ST_STM32G4:STM32G431CBTx
- J6: footprint Connector_PinHeader_2.54mm:PinHeader_1x05_P2.54mm_Vertical -> Connector_JST:JST_GH_BM05B-GHS-TBT_1x05-1MP_P1.25mm_Vertical; MPN (none) -> JST BM05B-GHS-TBT (1.25 mm, latching)
Connections:
- net +3V3: now also C35.1, C36.1, C37.1, C38.1, C39.1, U3.1 (VBAT), U3.24 (VDD), U3.36 (VDD), U3.48 (VDD)
- net +3V3A: now also C40.1, C41.1, U3.20 (VREF+), U3.21 (VDDA)
- net BOOT0: now also R26.1, U3.45 (PB8)
- net BRAKE: now also U3.3 (PC14)
- net DIR_SW: now also U3.34 (PA12)
- net GND: now also C35.2, C36.2, C37.2, C38.2, C39.2, C40.2, C41.2, C42.2, D6.1 (K), D7.1 (K), R26.2, U3.19 (VSSA), U3.23 (VSS), U3.35 (VSS), U3.47 (VSS)
- net HALL_A: now also U3.22 (PB10)
- net HALL_B: now also U3.25 (PB11)
- net HALL_C: now also U3.26 (PB12)
- net ISENSE_A: now also U3.8 (PA0)
- net ISENSE_B: now also U3.9 (PA1)
- net ISENSE_C: now also U3.10 (PA2)
- net LED_FAULT: now also R28.1, U3.18 (PB2)
- net LED_FAULT_A: now also D7.2 (A), R28.2
- net LED_STATUS: now also R27.1, U3.2 (PC13)
- net LED_STATUS_A: now also D6.2 (A), R27.2
- net NRST: now also C42.1, U3.7 (PG10)
- net PWM_AH: now also U3.30 (PA8)
- net PWM_AL: now also U3.27 (PB13)
- net PWM_BH: now also U3.31 (PA9)
- net PWM_BL: now also U3.28 (PB14)
- net PWM_CH: now also U3.32 (PA10)
- net PWM_CL: now also U3.29 (PB15)
- net PWR_BTN: now also U3.33 (PA11)
- net PWR_HOLD: now also U3.46 (PB9)
- net SWCLK: now also U3.38 (PA14)
- net SWDIO: now also U3.37 (PA13)
- net TEMP_FET: now also U3.13 (PA5)
- net TEMP_MOTOR: now also U3.14 (PA6)
- net THROTTLE: now also U3.12 (PA4)
- net UART_RX: now also U3.44 (PB7)
- net UART_TX: now also U3.43 (PB6)
- net VBUS_SENSE: now also U3.11 (PA3)
- new net DRV_CS: U3.39 (PA15)
- new net DRV_EN: U3.16 (PB0)
- new net DRV_FAULT: U3.17 (PB1)
- new net DRV_SCK: U3.40 (PB3)
- new net DRV_SDI: U3.42 (PB5)
- new net DRV_SDO: U3.41 (PB4)
- no-connect marks 10 -> 4
