File: hardware/kicad/power.kicad_sch (KiCad schematic)
At the start: 48 parts, among them J1 BAT+, J2 BAT-, Q1 MMBTA92, Q2 MMBTA42, U1 LM5164DDA, U2 LM5164DDA, U3 AP2112K-3.3

Commit message: Rev B: fix power terminals and design-review findings
Layout (hand-placed power stage):
- BAT+/BAT- and MOTOR A/B/C are now M5 plated bolt terminals at the board
  edges (battery 36 mm apart on the left edge, motors under their shunts),
  replacing 5x10 mm SMD solder pads that sat 7.5 mm apart
- per phase: driver | high FET over low FET (drain tabs up, compact switch
  node) | Kelvin shunt + INA240; DC-link ceramics at the low-side sources
- FET NTC moved next to the middle low-side FET
- rule area keeps tracks off the inner planes under the power stage
- pours sized from real TOLL pad outlines; solid plane connections
- hand route for the one connection Freerouting leaves open; routing
  session saved so the board rebuilds without the autorouter
- KiCad DRC: 0 violations, 0 unconnected, footprints match library

Schematic / firmware:
- INA240A2 -> INA240A1: the 80 A hard trip was above the old +/-66 A ADC
  full scale and could never fire; compile-time assert + sim test added
- 4-terminal Kelvin shunts (BVR 4026) feed the INA240 sense inputs
- gate resistors 10R -> 4R7, bulk caps 6 -> 8

Co-Authored-By: Claude Opus 5.5 <noreply@anthropic.com>
Claude-Session: https://claude.ai/code/session_01KE5bAkgcicsoh5erUtagKE
Parts:
- J1, J2: footprint Connector_Wire:SolderWirePad_1x01_SMD_5x10mm -> MountingHole:MountingHole_5.3mm_M5_Pad_Via; MPN (none) -> M5 ring lug terminal
Changed lines of the file:
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@@
     (rev "A")
     (company "48V 35A hub motor controller")
-    (comment 1 "STM32G431 + LM5109B x3 + IPT015N10N5 x6 + INA240A2 x3")
+    (comment 1 "STM32G431 + LM5109B x3 + IPT015N10N5 x6 + INA240A1 x3")
     (comment 2 "Sheet: power")
   )
@@
     (property "Reference" "J1" (at 35.29 28.21 0) (effects (font (size 1.27 1.27)) (justify left)))
     (property "Value" "BAT+" (at 35.29 33.75 0) (effects (font (size 1.27 1.27)) (justify left)))
-    (property "Footprint" "Connector_Wire:SolderWirePad_1x01_SMD_5x10mm" (at 33.02 30.48 0) (effects (font (size 1.27 1.27)) hide))
+    (property "Footprint" "MountingHole:MountingHole_5.3mm_M5_Pad_Via" (at 33.02 30.48 0) (effects (font (size 1.27 1.27)) hide))
     (property "Datasheet" "~" (at 33.02 30.48 0) (effects (font (size 1.27 1.27)) hide))
+    (property "MPN" "M5 ring lug terminal" (at 33.02 30.48 0) (effects (font (size 1.27 1.27)) hide))
     (pin "1")
     (instances (project "bldc48" (path "/1b798bf4-fe80-550a-af47-9df77e3c6d45/2f5e88aa-b08e-555a-ace0-10d8a5f9ef01" (reference "J1") (unit 1))))
@@
     (property "Reference" "J2" (at 58.15 28.21 0) (effects (font (size 1.27 1.27)) (justify left)))
     (property "Value" "BAT-" (at 58.15 33.75 0) (effects (font (size 1.27 1.27)) (justify left)))
-    (property "Footprint" "Connector_Wire:SolderWirePad_1x01_SMD_5x10mm" (at 55.88 30.48 0) (effects (font (size 1.27 1.27)) hide))
+    (property "Footprint" "MountingHole:MountingHole_5.3mm_M5_Pad_Via" (at 55.88 30.48 0) (effects (font (size 1.27 1.27)) hide))
     (property "Datasheet" "~" (at 55.88 30.48 0) (effects (font (size 1.27 1.27)) hide))
+    (property "MPN" "M5 ring lug terminal" (at 55.88 30.48 0) (effects (font (size 1.27 1.27)) hide))
     (pin "1")
     (instances (project "bldc48" (path "/1b798bf4-fe80-550a-af47-9df77e3c6d45/2f5e88aa-b08e-555a-ace0-10d8a5f9ef01" (reference "J2") (unit 1))))

Commit message: Rev C: compact 188x74 mm layout, re-routed, DRC clean; JLCPCB cost notes
- Repack the power stage into 38 mm phase columns and the logic into a 52 mm
  strip; smaller SRN8040TA buck inductors
- Re-route with Freerouting; record the LATCH_B hand route and move
  references that land on neighbouring silkscreen
- Regenerate BOM, schematic PDF, layer images and 3D renders (stand-in model
  for the SRN8040TA)
- README: rev C notes, phase-pour current capacity, JLCPCB cost estimate

Co-Authored-By: Claude Opus 5.5 <noreply@anthropic.com>
Claude-Session: https://claude.ai/code/session_01KE5bAkgcicsoh5erUtagKE
Parts:
- L1: footprint Inductor_SMD:L_Bourns_SRR1260 -> Inductor_SMD:L_Bourns_SRN8040TA; MPN SRR1260-680M -> Bourns SRN8040TA-680M or eq. (68 uH, Isat >= 0.8 A, 8x8 mm)
- L2: footprint Inductor_SMD:L_Bourns_SRR1260 -> Inductor_SMD:L_Bourns_SRN8040TA; MPN SRR1260-330M -> Bourns SRN8040TA-330M or eq. (33 uH, Isat >= 1 A, 8x8 mm)
Changed lines of the file:
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@@
     (property "Reference" "L1" (at 39.1 84.09 0) (effects (font (size 1.27 1.27)) (justify left)))
     (property "Value" "68u" (at 39.1 94.71 0) (effects (font (size 1.27 1.27)) (justify left)))
-    (property "Footprint" "Inductor_SMD:L_Bourns_SRR1260" (at 38.1 88.9 0) (effects (font (size 1.27 1.27)) hide))
+    (property "Footprint" "Inductor_SMD:L_Bourns_SRN8040TA" (at 38.1 88.9 0) (effects (font (size 1.27 1.27)) hide))
     (property "Datasheet" "~" (at 38.1 88.9 0) (effects (font (size 1.27 1.27)) hide))
-    (property "MPN" "SRR1260-680M" (at 38.1 88.9 0) (effects (font (size 1.27 1.27)) hide))
+    (property "MPN" "Bourns SRN8040TA-680M or eq. (68 uH, Isat >= 0.8 A, 8x8 mm)" (at 38.1 88.9 0) (effects (font (size 1.27 1.27)) hide))
     (pin "1")
     (pin "2")
@@
     (property "Reference" "L2" (at 232.14 84.09 0) (effects (font (size 1.27 1.27)) (justify left)))
     (property "Value" "33u" (at 232.14 94.71 0) (effects (font (size 1.27 1.27)) (justify left)))
-    (property "Footprint" "Inductor_SMD:L_Bourns_SRR1260" (at 231.14 88.9 0) (effects (font (size 1.27 1.27)) hide))
+    (property "Footprint" "Inductor_SMD:L_Bourns_SRN8040TA" (at 231.14 88.9 0) (effects (font (size 1.27 1.27)) hide))
     (property "Datasheet" "~" (at 231.14 88.9 0) (effects (font (size 1.27 1.27)) hide))
-    (property "MPN" "SRR1260-330M" (at 231.14 88.9 0) (effects (font (size 1.27 1.27)) hide))
-    (pin "1")
-    (pin "2")
+    (property "MPN" "Bourns SRN8040TA-330M or eq. (33 uH, Isat >= 1 A, 8x8 mm)" (at 231.14 88.9 0) (effects (font (size 1.27 1.27)) hide))
+    (pin "1")
+    (pin "2")

Commit message: BOM: LCSC part numbers, replacements for unstocked parts; revise cost
Bulk 220 uF/100 V caps are not stocked at LCSC: buy separately or use global
sourcing. Add a stocked alternative for the 33 uH inductor. Fix the cost
total (the low end did not match the sum of the rows).

Co-Authored-By: Claude Opus 5.5 <noreply@anthropic.com>
Claude-Session: https://claude.ai/code/session_01KE5bAkgcicsoh5erUtagKE
Parts:
- L1: MPN Bourns SRN8040TA-680M or eq. (68 uH, Isat >= 0.8 A, 8x8 mm) -> Bourns SRN8040TA-680M (LCSC C2047059)
- L2: MPN Bourns SRN8040TA-330M or eq. (33 uH, Isat >= 1 A, 8x8 mm) -> Bourns SRN8040TA-330M, or YJYCOIN YNR8040-330M (LCSC C49784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
Changed lines of the file:
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@@
     (property "Footprint" "Inductor_SMD:L_Bourns_SRN8040TA" (at 38.1 88.9 0) (effects (font (size 1.27 1.27)) hide))
     (property "Datasheet" "~" (at 38.1 88.9 0) (effects (font (size 1.27 1.27)) hide))
-    (property "MPN" "Bourns SRN8040TA-680M or eq. (68 uH, Isat >= 0.8 A, 8x8 mm)" (at 38.1 88.9 0) (effects (font (size 1.27 1.27)) hide))
+    (property "MPN" "Bourns SRN8040TA-680M (LCSC C2047059)" (at 38.1 88.9 0) (effects (font (size 1.27 1.27)) hide))
     (pin "1")
     (pin "2")
@@
     (property "Footprint" "Inductor_SMD:L_Bourns_SRN8040TA" (at 231.14 88.9 0) (effects (font (size 1.27 1.27)) hide))
     (property "Datasheet" "~" (at 231.14 88.9 0) (effects (font (size 1.27 1.27)) hide))
-    (property "MPN" "Bourns SRN8040TA-330M or eq. (33 uH, Isat >= 1 A, 8x8 mm)" (at 231.14 88.9 0) (effects (font (size 1.27 1.27)) hide))
-    (pin "1")
-    (pin "2")
+    (property "MPN" "Bourns SRN8040TA-330M, or YJYCOIN YNR8040-330M (LCSC C497847); 33 uH, Isat >= 1 A, 8x8 mm" (at 231.14 88.9 0) (effects (font (size 1.27 1.27)) hide))
+    (pin "1")
+    (pin "2")

Commit message: Rev F (in progress): DRV8353RS redesign for a 90 x 64.5 mm board
- Circuit: DRV8353RS gate driver + CSAs + 5 V buck replaces 3x LM5109B,
  3x INA240 and both LM5164s; low-side Kelvin shunts; 12 AWG solder-wire
  pads; JST-GH connectors; 3x 1000 uF bulk caps; project symbol/footprint
  library (DRV8353RS symbol + TI RGZ footprint from flatmcu, MIT)
- Firmware: SPI1 driver for the DRV8353 (config + readback + lock, fault
  readout, 'drv' command), ADC sampling at the PWM peak via TIM1 TRGO2,
  high-duty phase rebuilt from the other two, DRIVER fault; sim models the
  low-side shunt blind window and a driver fault - all checks pass
- Placement for the two-sided 3-column layout; router keepouts, pours and
  planes for it (board file stays rev E until routing is done)

Co-Authored-By: Claude Opus 5.5 <noreply@anthropic.com>
Claude-Session: https://claude.ai/code/session_01KE5bAkgcicsoh5erUtagKE
Parts:
- removed C11: 100n/100V, Capacitor_SMD:C_0805_2012Metric, symbol Device:C
- removed C12: 2.2n, Capacitor_SMD:C_0603_1608Metric, symbol Device:C
- removed C13: 3.3n, Capacitor_SMD:C_0603_1608Metric, symbol Device:C
- removed C14: 100n, Capacitor_SMD:C_0603_1608Metric, symbol Device:C
- removed C15, C16: 22u/10V, Capacitor_SMD:C_1210_3225Metric, symbol Device:C
- removed C17: 1u, Capacitor_SMD:C_0603_1608Metric, symbol Device:C
- removed C18: 4.7u, Capacitor_SMD:C_0805_2012Metric, symbol Device:C
- removed L2: 33u, Inductor_SMD:L_Bourns_SRN8040TA, symbol Device:L
- removed R13: 41.2k, Resistor_SMD:R_0603_1608Metric, symbol Device:R
- removed R14: 31.6k, Resistor_SMD:R_0603_1608Metric, symbol Device:R
- removed R15: 10k, Resistor_SMD:R_0603_1608Metric, symbol Device:R
- removed R16: 178k, Resistor_SMD:R_0603_1608Metric, symbol Device:R
- removed R17: 2.2k, Resistor_SMD:R_0603_1608Metric, symbol Device:R
- removed U2: LM5164DDA, Package_SO:HSOP-8-1EP_3.9x4.9mm_P1.27mm_EP2.41x3.1mm_ThermalVias, symbol Regulator_Switching:LM5164DDA
- removed U3: AP2112K-3.3, Package_TO_SOT_SMD:SOT-23-5, symbol Regulator_Linear:AP2112K-3.3
- added D5: GREEN, LED_SMD:LED_0603_1608Metric, symbol Device:LED
- C10: value 2.2u/100V -> 4.7u; footprint Capacitor_SMD:C_1210_3225Metric -> Capacitor_SMD:C_0805_2012Metric
- C2: value 1n -> 1u/100V; footprint Capacitor_SMD:C_0603_1608Metric -> Capacitor_SMD:C_0805_2012Metric
- C3: value 2.2u/100V -> 10n; footprint Capacitor_SMD:C_1210_3225Metric -> Capacitor_SMD:C_0603_1608Metric
- C4: value 100n/100V -> 1u; footprint Capacitor_SMD:C_0805_2012Metric -> Capacitor_SMD:C_0603_1608Metric
- C5: value 2.2n -> 47n
- C6: value 3.3n -> 330p
- C7: value 100n -> 22u/10V; footprint Capacitor_SMD:C_0603_1608Metric -> Capacitor_SMD:C_1210_3225Metric
- C8: value 22u/25V -> 4.7u; footprint Capacitor_SMD:C_1210_3225Metric -> Capacitor_SMD:C_0805_2012Metric
- C9: value 22u/25V -> 1u; footprint Capacitor_SMD:C_1210_3225Metric -> Capacitor_SMD:C_0603_1608Metric
- D4: value GREEN -> SS110; footprint LED_SMD:LED_0603_1608Metric -> Diode_SMD:D_SMA; symbol Device:LED -> Device:D; MPN (none) -> 100 V 1 A Schottky, SMA (e.g. MDD SS110)
- J1, J2: footprint MountingHole:MountingHole_5.3mm_M5_Pad_Via -> bldc48:SolderWire_12AWG_D2.8mm_OD5.4mm; MPN M5 ring lug terminal -> 12 AWG wire, soldered
- L1: value 68u -> 100u; footprint Inductor_SMD:L_Bourns_SRN8040TA -> Inductor_SMD:L_Bourns_SRN6045TA; MPN Bourns SRN8040TA-680M (LCSC C2047059) -> Bourns SRN6045TA-101M or eq. (100 uH, Isat >= 0.5 A, 6x6 mm)
- R10: value 90.9k -> 4.02k
- R11: value 10k -> 8.2k
- R12: value 365k -> 2.2k
- R7: value 330k -> 150k
- R8: value 27k -> 100k
- R9: value 100k -> 4.02k
- U1: value LM5164DDA -> AP2112K-3.3; footprint Package_SO:HSOP-8-1EP_3.9x4.9mm_P1.27mm_EP2.41x3.1mm_ThermalVias -> Package_TO_SOT_SMD:SOT-23-5; symbol Regulator_Switching:LM5164DDA -> Regulator_Linear:AP2112K-3.3
Connections:
- net +3V3: now also C10.1, R12.1, U1.5 (VOUT)
- net +48V: now also C2.1; no longer C10.1, C3.1, C4.1, U1.2 (VIN)
- net +5V: now also C5.2, C7.1, C8.1, C9.1, L1.2, R9.1, U1.1 (VIN), U1.3 (EN)
- net BST5: now also C3.1
- net FB5: now also C6.2, R10.1, R9.2
- net GND: now also C7.2, D4.2 (A), R10.2, U1.2 (GND), D5.1 (K); no longer C3.2, D4.1 (K), R11.2, R9.2, U1.1 (GND), U1.9 (EP)
- net PWR_LED_A: now also R12.2, D5.2 (A); no longer D4.2 (A)
- net RIP5: now also C5.1, C6.1, R11.2
- net SW5: now also C3.2, D4.1 (K), L1.1, R11.1
- removed net +12V: C6.2, C8.1, C9.1, L1.2, R10.1
- removed net BST12: C5.1, U1.7 (BST)
- removed net BUCK_EN: C2.1, R7.2, R8.1, U1.3 (EN/UVLO)
- removed net FB12: C7.2, R10.2, R11.1, U1.5 (FB)
- removed net RIP12: C6.1, C7.1, R12.2
- net RON12: no longer names the net of U1.4 (NC)
- net RON12: no longer R9.1
- removed net SW12: C5.2, L1.1, R12.1, U1.8 (SW)
- new net RCL: R8.1
- new net RT_SD: R7.2
- new net VCC_B: C4.1
- no-connect marks 2 -> 0
Other:
- note added: "Power input, soft-latch, 5 V buck, 3.3 V LDO"
- note removed: "Power input, soft-latch, supplies"
- title: Power input, soft-latch, supplies -> Power input, soft-latch, 5 V buck, 3.3 V LDO
- moved on the sheet: C10, C2, C3, C4, C5, C6, C7, C8, C9, L1, R10, R11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
